File: hardware/Digital IO Card/DigitalIODriver.kicad_sch (KiCad schematic)
At the start: 23 parts, among them Q1 RVQ040N05, Q2 RVQ040N05, Q3 2N7002, Q4 2N7002, U1 RT9624CGQWA, U2 RT9624CGQWA, U3 LM311DR

Commit message: DIO card initial schematic done
Parts:
- removed D1, D2: BAT54W, Package_TO_SOT_SMD:SOT-323_SC-70, symbol Diode:BAT54W
- added C12: 100nF, Capacitor_SMD:C_0603_1608Metric, symbol Device:C_Small
- added Q6: 2N7002, Package_TO_SOT_SMD:SOT-23, symbol Transistor_FET:2N7002
- added R12: 150, Resistor_SMD:R_1206_3216Metric, symbol Device:R_US
- added R19, R24: 133k, Resistor_SMD:R_0603_1608Metric, symbol Device:R_Small_US
- added R20: 14.7k, Resistor_SMD:R_0603_1608Metric, symbol Device:R_Small_US
- added R25: 33.2k, Resistor_SMD:R_0603_1608Metric, symbol Device:R_Small_US
- added U9: LM358, Package_SO:TSSOP-8_3x3mm_P0.65mm, symbol Amplifier_Operational:LM358
- renumbered C2 to C11, C4 to C6, C1 to C7, C3 to C8, C10 to C9, D3 to D1, Q4 to Q10, Q1 to Q7, Q2 to Q8, Q3 to Q9, R6 to R13, R4 to R14, R1 to R16, R3 to R17, R5 to R18, R15 to R21, R2 to R22, R23 to R27, U3 to U5, U1 to U7, U2 to U8
Connections:
- net LM311_V+ is gone; now on net +5V: C6.1, U5.8 (V+)
- net +5V: now also R13.2, R12.1
- net DIO: now also U9.3 (+); no longer R18.1
- net GND: now also C12.2, Q6.3 (D), R20.2, R25.2, U9.4 (V-)
- net V_{LOGIC}: now also C12.1, R19.1, U9.8 (V+); no longer R13.2
- net DIG_IN: now reaches R13.1, R14.1, U5.7
- net DIG_IN: now also Q6.1 (G)
- net at D1.1 (K): now also Q6.2 (S)
- net at D1.2 (A): now also R12.2
- net V_{LOGIC}/2 renamed V_{LOGIC}/10
- net V_{LOGIC}/10: now also R19.2, R20.1
- new net: R24.2, R25.1, U9.5 (+)
- new net DIO_BUFFERED: R24.1, U9.1, U9.2 (-)
- new net DIO/5: R18.1, U9.6 (-), U9.7
Other:
- note added: "Analog Level Shifter"
- note added: "HackerDAQ Digital I/O Driver"
- note added: "Schmitt Trigger Comparator"
- note added: "Status LED"
- note added: "This sheet implements the digital I/O driver for HackerDAQ. It is designed to power small DC loads such as relays, lights, and other electronics that need a DC input signal. It implements the following features: - Adjustable logic high voltage (V_{LOGIC}) between 3.3V and 24V - High current drive capability (up to 4A, if the power supply is sufficient) - Optional 10k pullup or pulldown - Status L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"
- note removed: "Logic Input Comparator"
- moved on the sheet: C11, C6, C7, C8, C9, D1, Q10, Q7, Q8, Q9, R13, R14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
