File: hardware/Digital IO Card/IOExpander.kicad_sch (KiCad schematic)
At the start: 2 parts, among them U34 MCP23S17_SS

Commit message: Start redoing DIO card
Parts:
- removed C51: 100nF, Capacitor_SMD:C_0603_1608Metric, symbol Device:C_Small
- removed U34: MCP23S17_SS, Package_SO:SSOP-28_5.3x10.2mm_P0.65mm, symbol Interface_Expansion:MCP23S17_SS
Connections:
- no-connect marks 6 -> 0
Other:
- note removed: "MCP23S17 SPI I/O Expander"
- note removed: "This circuit implements enough I/O for one bank of digital front ends via an MCP23S17 16-bit I/O expander. This allows them to be controlled using SPI commands at a clock of up to 10MHz. Note that the expander is powered off of 5V in order to produce 5V I/O for the front ends."
- title: I/O Expander -> (none)
