File: hardware/Digital IO Card/HackerDAQ Digital IO Card.kicad_pcb (KiCad board)
At the start: 2 copper layers, 90 x 90 mm, 79 parts, among them J2 MiniFit_Jr_5569_08A2, J3 MiniFit_Jr_5569_08A2, J4 MiniFit_Jr_5569_08A2, J5 MiniFit_Jr_5569_08A2, J6 HEADER_3x1, J9 LD15S33E4GX00LF, U1 SRV05-4.TCT, U2 SRV05-4.TCT, U3 SRV05-4.TCT, U35 MCP23S17_SS, U38 SN74AHC1G125, U4 M95320-RMN6, U5 SRV05-4.TCT, U6 SN74ACT17PWR, U7 TXB0106PW, U8 SN74ACT17PWR, U9 SN74ACT17PWR

Commit message: Finish redesigned DIO card
Parts:
- added D3: SMF5.0A, Diode_SMD:D_SMF, F.Cu at (118.0, 119.0)
- moved C2 77.1 mm to (101.0, 83.5)
- moved R27 55.2 mm to (105.5, 81.5), turned to 90 degrees
- moved R26 52.0 mm to (107.5, 81.5), turned to -90 degrees
- moved R31 43.7 mm to (130.5, 81.0), turned to 90 degrees
- moved R12 43.1 mm to (128.0, 76.0)
- moved R18 42.6 mm to (128.0, 78.0), turned to 180 degrees
- moved R32 42.0 mm to (132.5, 81.0), turned to -90 degrees
- moved LG1 11.3 mm to (58.2, 108.9)
- moved U3 1.58 mm to (131.5, 77.0)
- turned R10 to -90 degrees
- turned R11 to -90 degrees
- turned R15 to -90 degrees
- turned R16 to -90 degrees
- turned R28 to -90 degrees
- turned R29 to -90 degrees
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- renumbered C50 to C4, C31 to C5, C52 to C6, C4 to C7, D9 to D1, D17 to D10, D8 to D11, D14 to D12, D7 to D13, D13 to D14, D6 to D15, D5 to D16, D4 to D17, D3 to D18, D2 to D19, D10 to D2, D1 to D20, D11 to D4, D16 to D5, D19 to D6, D15 to D7, D18 to D8, D12 to D9, J2 to J1, J3 to J2, J4 to J3, J5 to J4, J6 to J5, J9 to J6, R32 to R10, R33 to R11, R13 to R12, R2 to R13, R6 to R14, R18 to R15, R20 to R16, R10 to R17, R14 to R18, R3 to R19, R17 to R2, R4 to R20, R23 to R21, R25 to R22, R28 to R23, R7 to R24, R8 to R25, R12 to R26, R11 to R27, R22 to R28, R24 to R3, R15 to R31, R16 to R32, R26 to R33, R107 to R34, R106 to R35, R27 to R4, R19 to R6, R21 to R7, R9 to R8, R31 to R9, U2 to U1, U7 to U10, U38 to U11, U3 to U2, U5 to U3, U1 to U4, U8 to U5, U9 to U6, U6 to U7, U35 to U8, U4 to U9
Routing:
- net +5V: track 24.0 -> 151.0 mm, vias 0 -> 11
- net /IOExpander/PA3: track 0.00 -> 60.7 mm
- net /IOExpander/PA0: track 0.00 -> 56.7 mm, vias 0 -> 2
- net V_{LOGIC}: track 356.7 -> 410.2 mm, vias 2 -> 6
- net /IOExpander/PA1: track 0.00 -> 52.2 mm, vias 0 -> 2
- net /IOExpander/PA2: track 0.00 -> 52.1 mm, vias 0 -> 2
- net /IOExpander/PA7: track 0.00 -> 42.6 mm
- net Net-(D5-A): track 0.00 -> 40.4 mm, vias 0 -> 1
- net /IOExpander/PA5: track 0.00 -> 32.2 mm
- net Net-(D7-A): track 0.00 -> 32.1 mm, vias 0 -> 1
- net Net-(D14-A): track 0.00 -> 31.7 mm, vias 0 -> 1
- net /IOExpander/PA4: track 0.00 -> 31.3 mm
- net /IOExpander/PA6: track 0.00 -> 30.4 mm, vias 0 -> 2
- net Net-(D6-A): track 0.00 -> 30.2 mm, vias 0 -> 1
- net Net-(D12-A): track 0.00 -> 28.8 mm, vias 0 -> 1
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Other:
- board text added: "(1) V_{LOGIC}"
- board text added: "(2) V_{LOGIC}"
- board text added: "(3) GND"
- board text added: "(4) GND"
- board text added: "(5) I/O d"
- board text added: "(6) I/O c"
- board text added: "(7) I/O b"
- board text added: "(8) I/O a"
- board text added: "0"
- board text added: "1"
- board text added: "10"
- board text added: "11"
- board text added: "12"
- board text added: "13"
- board text added: "14"
- board text added: "15"
- board text added: "2"
- board text added: "3"
- board text added: "4"
- board text added: "5"
- board text added: "6"
- board text added: "7"
- board text added: "8"
- board text added: "9"
- board text added: "Connector Pinout (looking INTO the face of the top connector):"
- board text added: "Mates with Mini-Fit 5557 series (e.g. 39013085)"
- board text added: "V_{LOGIC} is the 3.3V or 5V logic supply, selected via jumper."
