File: hardware/Digital IO Card/HackerDAQ Digital IO Card.kicad_pcb (KiCad board)
At the start: 2 copper layers, 90 x 90 mm, 80 parts, among them J1 MiniFit_Jr_5569_08A2, J2 MiniFit_Jr_5569_08A2, J3 MiniFit_Jr_5569_08A2, J4 MiniFit_Jr_5569_08A2, J5 HEADER_3x1, J6 LD15S33E4GX00LF, U1 SRV05-4.TCT, U10 TXB0106PW, U11 SN74AHC1G125, U2 SRV05-4.TCT, U3 SRV05-4.TCT, U4 SRV05-4.TCT, U5 SN74ACT17PWR, U6 SN74ACT17PWR, U7 SN74ACT17PWR, U8 MCP23S17_SS, U9 M95320-RMN6

Commit message: Fix swapped pins on digital I/O card, add kibot job
Parts:
- renumbered C5 to C31, J6 to J9, U9 to U4, U4 to U9
Connections:
- J1 pad 5: /IO0 -> /IO15
- J1 pad 6: /IO1 -> /IO14
- J1 pad 7: /IO2 -> /IO13
- J1 pad 8: /IO3 -> /IO12
- J2 pad 5: /IO4 -> /IO11
- J2 pad 6: /IO5 -> /IO10
- J2 pad 7: /IO6 -> /IO9
- J2 pad 8: /IO7 -> /IO8
- J3 pad 5: /IO8 -> /IO7
- J3 pad 6: /IO9 -> /IO6
- J3 pad 7: /IO10 -> /IO5
- J3 pad 8: /IO11 -> /IO4
- J4 pad 5: /IO12 -> /IO3
- J4 pad 6: /IO13 -> /IO2
- J4 pad 7: /IO14 -> /IO1
- J4 pad 8: /IO15 -> /IO0
- R1 pad 2: /IO0 -> /IO15
- R12 pad 2: /IO12 -> /IO3
- R13 pad 1: /IO1 -> /IO14
- R14 pad 1: /IO5 -> /IO10
- R17 pad 1: /IO9 -> /IO6
- R18 pad 1: /IO13 -> /IO2
- R19 pad 2: /IO2 -> /IO13
- R20 pad 1: /IO3 -> /IO12
- R24 pad 2: /IO6 -> /IO9
- R25 pad 1: /IO7 -> /IO8
- R26 pad 1: /IO11 -> /IO4
- R27 pad 2: /IO10 -> /IO5
- R31 pad 2: /IO14 -> /IO1
- R32 pad 1: /IO15 -> /IO0
- R5 pad 2: /IO4 -> /IO11
- R8 pad 2: /IO8 -> /IO7
- U1 pad 1: /IO5 -> /IO10
- U1 pad 3: /IO4 -> /IO11
- U1 pad 4: /IO6 -> /IO9
- U1 pad 6: /IO7 -> /IO8
- U2 pad 1: /IO9 -> /IO6
- U2 pad 3: /IO8 -> /IO7
- U2 pad 4: /IO10 -> /IO5
- U2 pad 6: /IO11 -> /IO4
- U3 pad 1: /IO13 -> /IO2
- U3 pad 3: /IO12 -> /IO3
- U3 pad 4: /IO14 -> /IO1
- U3 pad 6: /IO15 -> /IO0
- U9 pad 1: /IO1 -> /IO14
- U9 pad 3: /IO0 -> /IO15
- U9 pad 4: /IO2 -> /IO13
- U9 pad 6: /IO3 -> /IO12
Routing:
- net /IO4: track 9.45 -> 12.7 mm
- net /IO11: track 12.7 -> 9.45 mm
- net /IO3: track 13.9 -> 10.7 mm
- net /IO12: track 10.7 -> 13.9 mm
- net /IO8: track 10.3 -> 13.0 mm
- net /IO7: track 13.0 -> 10.3 mm
- net /IO15: track 11.6 -> 9.73 mm
- net /IO0: track 9.73 -> 11.6 mm
- net /IO2: track 13.9 -> 12.3 mm
- net /IO13: track 12.3 -> 13.9 mm
- net /IO5: track 11.6 -> 12.4 mm, vias 0 -> 2
- net /IO10: track 12.4 -> 11.6 mm, vias 2 -> 0
- net /IO9: track 12.1 -> 11.9 mm, vias 0 -> 2
- net /IO6: track 11.9 -> 12.1 mm, vias 2 -> 0

Commit message: Fix DRC/ERC errors
Parts:
- renumbered C2 to C1, C1 to C2, C31 to C5, J9 to J6, R6 to R1, R5 to R10, R8 to R11, R14 to R13, R17 to R14, R18 to R15, R13 to R16, R15 to R17, R16 to R18, R28 to R19, R7 to R2, R29 to R20, R30 to R21, R21 to R22, R22 to R23, R23 to R24, R24 to R25, R25 to R26, R26 to R28, R31 to R29, R9 to R3, R32 to R30, R19 to R31, R20 to R32, R10 to R4, R11 to R5, R1 to R6, R2 to R7, R3 to R8, R4 to R9, U9 to U1, U11 to U10, U10 to U11, U1 to U2, U2 to U3, U3 to U4, U7 to U6, U6 to U7, U4 to U9
