File: hardware/Digital IO Card/HackerDAQ Digital IO Card.kicad_sch (KiCad schematic)
At the start: 4 parts, among them J1 MiniFit_Jr_5569_08A2, J2 MiniFit_Jr_5569_08A2, J3 MiniFit_Jr_5569_08A2

Commit message: DIO card initial schematic done
Connections:
- net GND: now also J2.1 (Pin_1), J2.2 (Pin_2), J2.3 (Pin_3), J2.4 (Pin_4), J3.1 (Pin_1), J3.2 (Pin_2), J3.3 (Pin_3), J3.4 (Pin_4)
- net DIOA0: now reaches J2.5 (Pin_5)
- net DIOA1: now reaches J2.6 (Pin_6)
- net DIOA2: now reaches J2.7 (Pin_7)
- net DIOA3: now reaches J2.8 (Pin_8)
- net DIOB0: now reaches J3.5 (Pin_5)
- net DIOB1: now reaches J3.6 (Pin_6)
- net DIOB2: now reaches J3.7 (Pin_7)
- net DIOB3: now reaches J3.8 (Pin_8)
- net VLOGIC_BANK0 renamed V_{LOGIC}_PORTA
- net VLOGIC_BANK1 renamed V_{LOGIC}_PORTB
- no-connect marks 1 -> 4
Other:
- sheet DigitalIODriver0 renamed DigitalIODriverA0
- added sheet DigitalIODriverA1 (DigitalIODriver.kicad_sch)
- added sheet DigitalIODriverA2 (DigitalIODriver.kicad_sch)
- added sheet DigitalIODriverA3 (DigitalIODriver.kicad_sch)
- added sheet DigitalIODriverB0 (DigitalIODriver.kicad_sch)
- added sheet DigitalIODriverB1 (DigitalIODriver.kicad_sch)
- added sheet DigitalIODriverB2 (DigitalIODriver.kicad_sch)
- added sheet DigitalIODriverB3 (DigitalIODriver.kicad_sch)
- added sheet IOExpanderA (IOExpander.kicad_sch)
- added sheet IOExpanderB (IOExpander.kicad_sch)
- added sheet LevelShifter (LevelShifter.kicad_sch)
- sheet DigitalIODriverA0 ports: added DIG_IN, DIO, HICUR_LOGIC_CTRL, PULL_LOGIC_CTRL, V_{LOGIC}; removed none
- sheet SPI EEPROM ports: added V_{CC}; removed none
- note added: "Digital Front Ends (Port A)"
- note added: "Digital Front Ends (Port B)"
- note added: "I/O Expanders"
- note added: "Identity EEPROM"
- note added: "Main Board Interface"
- note added: "V_{LOGIC} Selection"
- moved on the sheet: J1, J3, LG1

Commit message: Start redoing DIO card
Parts:
- removed J1: MiniFit_Jr_5569_08A2, Project Library:Molex_Mini-Fit_Jr_5569-08A2_2x04_P4.20mm_Horizontal, symbol Project Library:MiniFit_Jr_5569_08A2
- added D1, D12, D13, D14, D15, D16, D17, D18, D19, D2, D3, D4, D5, D6, D7, D8: AA3528SURSK, ColorLEDs:AA3528, symbol ColorLEDs:AA3528SURSK
- added J4, J5: MiniFit_Jr_5569_08A2, Project Library:Molex_Mini-Fit_Jr_5569-08A2_2x04_P4.20mm_Horizontal, symbol Project Library:MiniFit_Jr_5569_08A2
- added J6: HEADER_3x1, Connector_PinHeader_2.54mm:PinHeader_1x03_P2.54mm_Vertical, symbol Connector:Conn_01x03_Pin
- added M1: QPC02SXGN-RC, symbol Project Library:Jumper
- added R17, R18, R19, R20, R21, R22, R23, R24, R25, R27, R28, R29, R30, R31, R32, R33: 150, Resistor_SMD:R_1206_3216Metric, symbol Device:R_US
Connections:
- net +3.3V: now also J6.3 (Pin_3)
- net +5V: now also J6.1 (Pin_1)
- net GND: now also D1.1 (K), D12.1 (K), D13.1 (K), D14.1 (K), D15.1 (K), D16.1 (K), D17.1 (K), D18.1 (K), D19.1 (K), D2.1 (K), D3.1 (K), D4.1 (K), D5.1 (K), D6.1 (K), D7.1 (K), D8.1 (K), J4.3 (Pin_3), J4.4 (Pin_4), J5.3 (Pin_3), J5.4 (Pin_4); no longer J2.1 (Pin_1), J2.2 (Pin_2), J3.1 (Pin_1), J3.2 (Pin_2)
- net DIOA0 renamed IO0
- net DIOA1 renamed IO1
- net DIOA2 renamed IO2
- net DIOA3 renamed IO3
- net DIOB0 renamed IO4
- net DIOB1 renamed IO5
- net DIOB2 renamed IO6
- net DIOB3 renamed IO7
- new net: D13.2 (A), R18.1
- new net: D1.2 (A), R17.1
- new net: D3.2 (A), R24.1
- new net: D18.2 (A), R32.1
- new net: D16.2 (A), R30.1
- new net: D4.2 (A), R25.1
- new net: D8.2 (A), R21.1
- new net: D17.2 (A), R31.1
- new net: D2.2 (A), R23.1
- new net: D7.2 (A), R19.1
- new net: D5.2 (A), R27.1
- new net: D15.2 (A), R29.1
- new net: D6.2 (A), R28.1
- new net: D19.2 (A), R33.1
- new net: D14.2 (A), R20.1
- new net: D12.2 (A), R22.1
- new net IO0_LED: R17.2
- new net IO10: J4.7 (Pin_7)
- new net IO10_LED: R31.2
- new net IO11: J4.8 (Pin_8)
- new net IO11_LED: R22.2
- new net IO12: J5.5 (Pin_5)
- new net IO12_LED: R32.2
- new net IO13: J5.6 (Pin_6)
- new net IO13_LED: R29.2
- new net IO14: J5.7 (Pin_7)
- new net IO14_LED: R33.2
- new net IO15: J5.8 (Pin_8)
- new net IO15_LED: R30.2
- new net IO1_LED: R23.2
- new net IO2_LED: R24.2
- new net IO3_LED: R25.2
- new net IO4_LED: R27.2
- new net IO5_LED: R28.2
- new net IO6_LED: R18.2
- new net IO7_LED: R19.2
- new net IO8: J4.5 (Pin_5)
- new net IO8_LED: R20.2
- new net IO9: J4.6 (Pin_6)
- new net IO9_LED: R21.2
- new net V_{LOGIC}: J2.1 (Pin_1), J2.2 (Pin_2), J3.1 (Pin_1), J3.2 (Pin_2), J4.1 (Pin_1), J4.2 (Pin_2), J5.1 (Pin_1), J5.2 (Pin_2), J6.2 (Pin_2)
- no-connect marks 4 -> 6
Other:
- sheet IOExpanderA renamed IOExpander
- removed sheet DigitalIODriverA0
- removed sheet DigitalIODriverA1
- removed sheet DigitalIODriverA2
- removed sheet DigitalIODriverA3
- removed sheet DigitalIODriverB0
- removed sheet DigitalIODriverB1
- removed sheet DigitalIODriverB2
- removed sheet DigitalIODriverB3
- removed sheet IOExpanderB
- added sheet IOProtection0 (IOProtection.kicad_sch)
- added sheet IOProtection1 (IOProtection.kicad_sch)
- added sheet IOProtection2 (IOProtection.kicad_sch)
- added sheet IOProtection3 (IOProtection.kicad_sch)
- added sheet LEDDriver0 (LEDDriver.kicad_sch)
- added sheet LEDDriver1 (LEDDriver.kicad_sch)
- added sheet LEDDriver2 (LEDDriver.kicad_sch)
- sheet IOExpander: file IOExpander.kicad_sch -> ../Common Sheets/IOExpander.kicad_sch
- sheet IOExpander ports: added PA[0..7], PB[0..7], SPI{MOSI MISO SCLK}, V_{DD}; removed DIG_IN[0..3], HICUR_LOGIC_CTRL[0..3], PULL_LOGIC_CTRL[0..3], SPI_5V{MOSI MISO SCLK}
- sheet LevelShifter ports: added SPI_VL{MOSI MISO SCLK}, ~{CS_VL}[0..2], ~{RESET_VL}; removed SPI_5V{MOSI MISO SCLK}, ~{CS_5V}[0..2], ~{RESET_5V}
- note added: "I/O Expander"
- note added: "I/O Ports"
- note removed: "Digital Front Ends (Port A)"
- note removed: "Digital Front Ends (Port B)"
- note removed: "I/O Expanders"
- moved on the sheet: J2

Commit message: Finish redesigned DIO card
Parts:
- added D20: SMF5.0A, Diode_SMD:D_SMF, symbol Diode:SMF11A
- renumbered D8 to D10, D14 to D11, D7 to D12, D6 to D14, D5 to D15, D4 to D16, D3 to D17, D2 to D18, D1 to D19, D16 to D4, D19 to D5, D15 to D6, D18 to D7, D12 to D8, D17 to D9, J2 to J1, J3 to J2, J4 to J3, J5 to J4, J6 to J5, R32 to R10, R33 to R11, R18 to R15, R20 to R16, R17 to R2, R23 to R21, R25 to R22, R28 to R23, R22 to R28, R24 to R3, R27 to R4, R19 to R6, R21 to R7, R31 to R9
Connections:
- net GND: now also D20.2 (A2)
- net V_{LOGIC}: now also D20.1 (A1)

Commit message: Back-annotate
Parts:
- renumbered D9 to D10, D10 to D11, D11 to D12, D12 to D13, D13 to D14, D14 to D15, D15 to D16, D16 to D17, D17 to D18, D18 to D19, D19 to D20, D20 to D3, D4 to D5, D5 to D6, D6 to D7, D7 to D8, D8 to D9
Changed lines of the file:
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@@
 		(on_board yes)
 		(dnp no)
-		(property "Reference" "D4"
+		(property "Reference" "D5"
 			(at 67.056 175.26 0)
 			(effects
@@
 			(project "HackerDAQ Digital IO Card"
 				(path "/af2d881c-6553-449d-9093-6deb41497bdc"
-					(reference "D4")
+					(reference "D5")
 					(unit 1)
 				)
@@
 		(on_board yes)
 		(dnp no)
-		(property "Reference" "D10"
+		(property "Reference" "D11"
 			(at 68.326 123.19 0)
 			(effects
@@
 			(project "HackerDAQ Digital IO Card"
 				(path "/af2d881c-6553-449d-9093-6deb41497bdc"
-					(reference "D10")
+					(reference "D11")
 					(unit 1)
 				)
@@
 		(on_board yes)
 		(dnp no)
-		(property "Reference" "D9"
+		(property "Reference" "D10"
 			(at 74.422 161.798 0)
 			(effects
@@
 			(project "HackerDAQ Digital IO Card"
 				(path "/af2d881c-6553-449d-9093-6deb41497bdc"
-					(reference "D9")
+					(reference "D10")
 					(unit 1)
 				)
@@
 		(on_board yes)
 		(dnp no)
-		(property "Reference" "D12"
+		(property "Reference" "D13"
 			(at 68.326 117.602 0)
 			(effects
@@
 			(project "HackerDAQ Digital IO Card"
 				(path "/af2d881c-6553-449d-9093-6deb41497bdc"
-					(reference "D12")
+					(reference "D13")
 					(unit 1)
 				)
@@
 		(on_board yes)
 		(dnp no)
-		(property "Reference" "D14"
+		(property "Reference" "D15"
 			(at 68.326 74.93 0)
 			(effects
@@
 			(project "HackerDAQ Digital IO Card"
 				(path "/af2d881c-6553-449d-9093-6deb41497bdc"
-					(reference "D14")
+					(reference "D15")
 					(unit 1)
 				)
@@
 		(on_board yes)
 		(dnp no)
-		(property "Reference" "D5"
+		(property "Reference" "D6"
 			(at 80.264 172.466 0)
 			(effects
@@
 			(project "HackerDAQ Digital IO Card"
 				(path "/af2d881c-6553-449d-9093-6deb41497bdc"
-					(reference "D5")
+					(reference "D6")
 					(unit 1)
 				)
@@
 		(on_board yes)
 		(dnp no)
-		(property "Reference" "D11"
+		(property "Reference" "D12"
 			(at 81.534 120.396 0)
 			(effects
@@
 			(project "HackerDAQ Digital IO Card"
 				(path "/af2d881c-6553-449d-9093-6deb41497bdc"
-					(reference "D11")
+					(reference "D12")
 					(unit 1)
 				)
@@
 		(on_board yes)
 		(dnp no)
-		(property "Reference" "D16"
+		(property "Reference" "D17"
 			(at 68.326 69.85 0)
 			(effects
@@
 			(project "HackerDAQ Digital IO Card"
 				(path "/af2d881c-6553-449d-9093-6deb41497bdc"
-					(reference "D16")
+					(reference "D17")
 					(unit 1)
 				)
@@
 		(on_board yes)
 		(dnp no)
-		(property "Reference" "D18"
+		(property "Reference" "D19"
 			(at 68.326 64.262 0)
 			(effects
@@
 			(project "HackerDAQ Digital IO Card"
 				(path "/af2d881c-6553-449d-9093-6deb41497bdc"
-					(reference "D18")
+					(reference "D19")
 					(unit 1)
 				)
@@
 		(on_board yes)
 		(dnp no)
-		(property "Reference" "D19"
+		(property "Reference" "D20"
 			(at 75.692 61.468 0)
 			(effects
@@
 			(project "HackerDAQ Digital IO Card"
 				(path "/af2d881c-6553-449d-9093-6deb41497bdc"
-					(reference "D19")
+					(reference "D20")
 					(unit 1)
 				)
@@
 		(on_board yes)
 		(dnp no)
-		(property "Reference" "D6"
+		(property "Reference" "D7"
 			(at 67.056 170.18 0)
 			(effects
@@
 			(project "HackerDAQ Digital IO Card"
 				(path "/af2d881c-6553-449d-9093-6deb41497bdc"
-					(reference "D6")
+					(reference "D7")
 					(unit 1)
 				)
@@
 		(on_board yes)
 		(dnp no)
-		(property "Reference" "D17"
+		(property "Reference" "D18"
 			(at 81.534 67.056 0)
 			(effects
@@
 			(project "HackerDAQ Digital IO Card"
 				(path "/af2d881c-6553-449d-9093-6deb41497bdc"
-					(reference "D17")
+					(reference "D18")
 					(unit 1)
 				)
@@
 		(dnp no)
 		(fields_autoplaced yes)
-		(property "Reference" "D20"
+		(property "Reference" "D3"
 			(at 298.45 68.5799 90)
 			(effects
@@
 			(project "HackerDAQ Digital IO Card"
 				(path "/af2d881c-6553-449d-9093-6deb41497bdc"
-					(reference "D20")
+					(reference "D3")
 					(unit 1)
 				)
@@
 		(on_board yes)
 		(dnp no)
-		(property "Reference" "D7"
+		(property "Reference" "D8"
 			(at 80.264 167.386 0)
 			(effects
@@
 			(project "HackerDAQ Digital IO Card"
 				(path "/af2d881c-6553-449d-9093-6deb41497bdc"
-					(reference "D7")
+					(reference "D8")
 					(unit 1)
 				)
@@
 		(on_board yes)
 		(dnp no)
-		(property "Reference" "D13"
+		(property "Reference" "D14"
 			(at 75.692 114.808 0)
 			(effects
@@
 			(project "HackerDAQ Digital IO Card"
 				(path "/af2d881c-6553-449d-9093-6deb41497bdc"
-					(reference "D13")
+					(reference "D14")
 					(unit 1)
 				)
@@
 		(on_board yes)
 		(dnp no)
-		(property "Reference" "D8"
+		(property "Reference" "D9"
 			(at 67.056 164.592 0)
 			(effects
@@
 			(project "HackerDAQ Digital IO Card"
 				(path "/af2d881c-6553-449d-9093-6deb41497bdc"
-					(reference "D8")
+					(reference "D9")
 					(unit 1)
 				)
@@
 		(on_board yes)
 		(dnp no)
-		(property "Reference" "D15"
+		(property "Reference" "D16"
 			(at 81.534 72.136 0)
 			(effects
@@
 			(project "HackerDAQ Digital IO Card"
 				(path "/af2d881c-6553-449d-9093-6deb41497bdc"
-					(reference "D15")
+					(reference "D16")
 					(unit 1)
 				)
