File: hardware/Digital IO Card/HackerDAQ Digital IO Card.kicad_sch (KiCad schematic)
At the start: 40 parts, among them J1 MiniFit_Jr_5569_08A2, J2 MiniFit_Jr_5569_08A2, J3 MiniFit_Jr_5569_08A2, J4 MiniFit_Jr_5569_08A2, J5 HEADER_3x1, M1 QPC02SXGN-RC

Commit message: Fix swapped pins on digital I/O card, add kibot job
Connections:
- net IO0: now also J4.8 (Pin_8); no longer J1.5 (Pin_5)
- net IO1: now also J4.7 (Pin_7); no longer J1.6 (Pin_6)
- net IO10: now also J2.6 (Pin_6); no longer J3.7 (Pin_7)
- net IO11: now also J2.5 (Pin_5); no longer J3.8 (Pin_8)
- net IO12: now also J1.8 (Pin_8); no longer J4.5 (Pin_5)
- net IO13: now also J1.7 (Pin_7); no longer J4.6 (Pin_6)
- net IO14: now also J1.6 (Pin_6); no longer J4.7 (Pin_7)
- net IO15: now also J1.5 (Pin_5); no longer J4.8 (Pin_8)
- net IO2: now also J4.6 (Pin_6); no longer J1.7 (Pin_7)
- net IO3: now also J4.5 (Pin_5); no longer J1.8 (Pin_8)
- net IO4: now also J3.8 (Pin_8); no longer J2.5 (Pin_5)
- net IO5: now also J3.7 (Pin_7); no longer J2.6 (Pin_6)
- net IO6: now also J3.6 (Pin_6); no longer J2.7 (Pin_7)
- net IO7: now also J3.5 (Pin_5); no longer J2.8 (Pin_8)
- net IO8: now also J2.8 (Pin_8); no longer J3.5 (Pin_5)
- net IO9: now also J2.7 (Pin_7); no longer J3.6 (Pin_6)
Changed lines of the file:
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@@
 		)
 	)
-	(label "IO10"
+	(label "IO5"
 		(at 58.42 147.32 0)
 		(effects
@@
 		)
 	)
-	(label "IO8"
+	(label "IO7"
 		(at 58.42 142.24 0)
 		(effects
@@
 		)
 	)
-	(label "IO6"
+	(label "IO9"
 		(at 58.42 99.06 0)
 		(effects
@@
 		)
 	)
-	(label "IO7"
+	(label "IO8"
 		(at 58.42 101.6 0)
 		(effects
@@
 		)
 	)
-	(label "IO13"
+	(label "IO2"
 		(at 58.42 198.12 0)
 		(effects
@@
 		)
 	)
-	(label "IO5"
+	(label "IO10"
 		(at 58.42 96.52 0)
 		(effects
@@
 		)
 	)
-	(label "IO2"
+	(label "IO13"
 		(at 58.42 48.26 0)
 		(effects
@@
 		)
 	)
-	(label "IO15"
+	(label "IO0"
 		(at 58.42 203.2 0)
 		(effects
@@
 		)
 	)
-	(label "IO9"
+	(label "IO6"
 		(at 58.42 144.78 0)
 		(effects
@@
 		)
 	)
-	(label "IO4"
+	(label "IO11"
 		(at 58.42 93.98 0)
 		(effects
@@
 		)
 	)
-	(label "IO14"
+	(label "IO1"
 		(at 58.42 200.66 0)
 		(effects
@@
 		)
 	)
-	(label "IO11"
+	(label "IO4"
 		(at 58.42 149.86 0)
 		(effects
@@
 		)
 	)
-	(label "IO0"
+	(label "IO15"
 		(at 58.42 43.18 0)
 		(effects
@@
 		)
 	)
-	(label "IO1"
+	(label "IO14"
 		(at 58.42 45.72 0)
 		(effects
@@
 		)
 	)
-	(label "IO3"
+	(label "IO12"
 		(at 58.42 50.8 0)
 		(effects
@@
 		)
 	)
-	(label "IO12"
+	(label "IO3"
 		(at 58.42 195.58 0)
 		(effects

Commit message: Fix DRC/ERC errors
Parts:
- renumbered R6 to R1, R15 to R17, R16 to R18, R28 to R19, R7 to R2, R29 to R20, R30 to R21, R21 to R22, R22 to R23, R23 to R24, R9 to R3, R10 to R4, R11 to R5, R2 to R7, R3 to R8, R4 to R9
Changed lines of the file:
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@@
 		(on_board yes)
 		(dnp no)
-		(property "Reference" "R15"
+		(property "Reference" "R17"
 			(at 95.25 115.316 90)
 			(effects
@@
 			(project "HackerDAQ Digital IO Card"
 				(path "/af2d881c-6553-449d-9093-6deb41497bdc"
-					(reference "R15")
+					(reference "R17")
 					(unit 1)
 				)
@@
 		(on_board yes)
 		(dnp no)
-		(property "Reference" "R2"
+		(property "Reference" "R7"
 			(at 95.25 61.976 90)
 			(effects
@@
 			(project "HackerDAQ Digital IO Card"
 				(path "/af2d881c-6553-449d-9093-6deb41497bdc"
-					(reference "R2")
+					(reference "R7")
 					(unit 1)
 				)
@@
 		(on_board yes)
 		(dnp no)
-		(property "Reference" "R3"
+		(property "Reference" "R8"
 			(at 95.25 67.056 90)
 			(effects
@@
 			(project "HackerDAQ Digital IO Card"
 				(path "/af2d881c-6553-449d-9093-6deb41497bdc"
-					(reference "R3")
+					(reference "R8")
 					(unit 1)
 				)
@@
 		(on_board yes)
 		(dnp no)
-		(property "Reference" "R10"
+		(property "Reference" "R4"
 			(at 93.98 167.386 90)
 			(effects
@@
 			(project "HackerDAQ Digital IO Card"
 				(path "/af2d881c-6553-449d-9093-6deb41497bdc"
-					(reference "R10")
+					(reference "R4")
 					(unit 1)
 				)
@@
 		(on_board yes)
 		(dnp no)
-		(property "Reference" "R22"
+		(property "Reference" "R23"
 			(at 85.09 69.596 90)
 			(effects
@@
 			(project "HackerDAQ Digital IO Card"
 				(path "/af2d881c-6553-449d-9093-6deb41497bdc"
-					(reference "R22")
+					(reference "R23")
 					(unit 1)
 				)
@@
 		(on_board yes)
 		(dnp no)
-		(property "Reference" "R21"
+		(property "Reference" "R22"
 			(at 85.09 64.516 90)
 			(effects
@@
 			(project "HackerDAQ Digital IO Card"
 				(path "/af2d881c-6553-449d-9093-6deb41497bdc"
-					(reference "R21")
+					(reference "R22")
 					(unit 1)
 				)
@@
 		(on_board yes)
 		(dnp no)
-		(property "Reference" "R4"
+		(property "Reference" "R9"
 			(at 95.25 72.136 90)
 			(effects
@@
 			(project "HackerDAQ Digital IO Card"
 				(path "/af2d881c-6553-449d-9093-6deb41497bdc"
-					(reference "R4")
+					(reference "R9")
 					(unit 1)
 				)
@@
 		(on_board yes)
 		(dnp no)
-		(property "Reference" "R29"
+		(property "Reference" "R20"
 			(at 83.82 169.926 90)
 			(effects
@@
 			(project "HackerDAQ Digital IO Card"
 				(path "/af2d881c-6553-449d-9093-6deb41497bdc"
-					(reference "R29")
+					(reference "R20")
 					(unit 1)
 				)
@@
 		(on_board yes)
 		(dnp no)
-		(property "Reference" "R6"
+		(property "Reference" "R1"
 			(at 87.63 117.856 90)
 			(effects
@@
 			(project "HackerDAQ Digital IO Card"
 				(path "/af2d881c-6553-449d-9093-6deb41497bdc"
-					(reference "R6")
+					(reference "R1")
 					(unit 1)
 				)
@@
 		(on_board yes)
 		(dnp no)
-		(property "Reference" "R9"
+		(property "Reference" "R3"
 			(at 93.98 162.306 90)
 			(effects
@@
 			(project "HackerDAQ Digital IO Card"
 				(path "/af2d881c-6553-449d-9093-6deb41497bdc"
-					(reference "R9")
+					(reference "R3")
 					(unit 1)
 				)
@@
 		(on_board yes)
 		(dnp no)
-		(property "Reference" "R30"
+		(property "Reference" "R21"
 			(at 83.82 175.006 90)
 			(effects
@@
 			(project "HackerDAQ Digital IO Card"
 				(path "/af2d881c-6553-449d-9093-6deb41497bdc"
-					(reference "R30")
+					(reference "R21")
 					(unit 1)
 				)
@@
 		(on_board yes)
 		(dnp no)
-		(property "Reference" "R7"
+		(property "Reference" "R2"
 			(at 87.63 122.936 90)
 			(effects
@@
 			(project "HackerDAQ Digital IO Card"
 				(path "/af2d881c-6553-449d-9093-6deb41497bdc"
-					(reference "R7")
+					(reference "R2")
 					(unit 1)
 				)
@@
 		(on_board yes)
 		(dnp no)
-		(property "Reference" "R23"
+		(property "Reference" "R24"
 			(at 85.09 74.676 90)
 			(effects
@@
 			(project "HackerDAQ Digital IO Card"
 				(path "/af2d881c-6553-449d-9093-6deb41497bdc"
-					(reference "R23")
+					(reference "R24")
 					(unit 1)
 				)
@@
 		(on_board yes)
 		(dnp no)
-		(property "Reference" "R11"
+		(property "Reference" "R5"
 			(at 93.98 172.466 90)
 			(effects
@@
 			(project "HackerDAQ Digital IO Card"
 				(path "/af2d881c-6553-449d-9093-6deb41497bdc"
-					(reference "R11")
+					(reference "R5")
 					(unit 1)
 				)
@@
 		(on_board yes)
 		(dnp no)
-		(property "Reference" "R28"
+		(property "Reference" "R19"
 			(at 83.82 164.846 90)
 			(effects
@@
 			(project "HackerDAQ Digital IO Card"
 				(path "/af2d881c-6553-449d-9093-6deb41497bdc"
-					(reference "R28")
+					(reference "R19")
 					(unit 1)
 				)
@@
 		(on_board yes)
 		(dnp no)
-		(property "Reference" "R16"
+		(property "Reference" "R18"
 			(at 95.25 120.396 90)
 			(effects
@@
 			(project "HackerDAQ Digital IO Card"
 				(path "/af2d881c-6553-449d-9093-6deb41497bdc"
-					(reference "R16")
+					(reference "R18")
 					(unit 1)
 				)

Commit message: Add some docs
Other:
- note added: "HackerDAQ Digital I/O Card"
- note added: "This card provides 16 basic digital I/O lines from one slot of a HackerDAQ. It is fairly simple and most functionality is provided by an MCP23S17 I/O expander. Features: - 16x I/O lines, mappable as inputs or outputs - Selectable logic voltage, 3.3V or 5V - 3mA source / 8mA sink output current per line - ESD protection on I/O lines - High input impedance when in input mode (1.6MOhm or better) - S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"
- moved on the sheet: D10, D11, D12, D13, D14, D15, D16, D17, D18, D19, D20, D3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
