File: hardware/Digital IO Card/IOProtection.kicad_sch (KiCad schematic)
At the start: 5 parts, among them U2 SRV05-4.TCT

Commit message: Finish redesigned DIO card
Parts:
- renumbered R6 to R14, R7 to R24, R8 to R25, U2 to U1
Changed lines of the file:
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@@
 		(on_board yes)
 		(dnp no)
-		(property "Reference" "R6"
+		(property "Reference" "R14"
 			(at 93.726 48.006 90)
 			(effects
@@
 			(project "HackerDAQ Digital IO Card"
 				(path "/af2d881c-6553-449d-9093-6deb41497bdc/455d3721-42aa-4f0e-b48f-29a642ac1f78"
-					(reference "R2")
+					(reference "R13")
 					(unit 1)
 				)
 				(path "/af2d881c-6553-449d-9093-6deb41497bdc/67eb63b8-4985-495d-ab9e-4c58fb498c7d"
+					(reference "R18")
+					(unit 1)
+				)
+				(path "/af2d881c-6553-449d-9093-6deb41497bdc/777ce27f-f0db-4b38-a663-f213b2d41686"
 					(reference "R14")
 					(unit 1)
 				)
-				(path "/af2d881c-6553-449d-9093-6deb41497bdc/777ce27f-f0db-4b38-a663-f213b2d41686"
-					(reference "R6")
-					(unit 1)
-				)
 				(path "/af2d881c-6553-449d-9093-6deb41497bdc/97e743ff-8a82-4285-b0f3-f0e89ab922fa"
-					(reference "R10")
+					(reference "R17")
 					(unit 1)
 				)
@@
 		(on_board yes)
 		(dnp no)
-		(property "Reference" "R8"
+		(property "Reference" "R25"
 			(at 102.616 55.626 90)
 			(effects
@@
 			(project "HackerDAQ Digital IO Card"
 				(path "/af2d881c-6553-449d-9093-6deb41497bdc/455d3721-42aa-4f0e-b48f-29a642ac1f78"
-					(reference "R4")
+					(reference "R20")
 					(unit 1)
 				)
 				(path "/af2d881c-6553-449d-9093-6deb41497bdc/67eb63b8-4985-495d-ab9e-4c58fb498c7d"
-					(reference "R16")
+					(reference "R32")
 					(unit 1)
 				)
 				(path "/af2d881c-6553-449d-9093-6deb41497bdc/777ce27f-f0db-4b38-a663-f213b2d41686"
-					(reference "R8")
+					(reference "R25")
 					(unit 1)
 				)
 				(path "/af2d881c-6553-449d-9093-6deb41497bdc/97e743ff-8a82-4285-b0f3-f0e89ab922fa"
-					(reference "R12")
+					(reference "R26")
 					(unit 1)
 				)
@@
 		(dnp no)
 		(property "Reference" "R5"
-			(at 90.424 39.624 90)
+			(at 89.154 40.386 90)
 			(effects
 				(font
@@
 		)
 		(property "Value" "33"
-			(at 94.234 39.624 90)
+			(at 95.25 40.386 90)
 			(effects
 				(font
@@
 				)
 				(path "/af2d881c-6553-449d-9093-6deb41497bdc/67eb63b8-4985-495d-ab9e-4c58fb498c7d"
-					(reference "R13")
+					(reference "R12")
 					(unit 1)
 				)
@@
 				)
 				(path "/af2d881c-6553-449d-9093-6deb41497bdc/97e743ff-8a82-4285-b0f3-f0e89ab922fa"
-					(reference "R9")
+					(reference "R8")
 					(unit 1)
 				)
@@
 		(dnp no)
 		(fields_autoplaced yes)
-		(property "Reference" "U2"
+		(property "Reference" "U1"
 			(at 69.1581 63.5 0)
 			(effects
@@
 			(project "HackerDAQ Digital IO Card"
 				(path "/af2d881c-6553-449d-9093-6deb41497bdc/455d3721-42aa-4f0e-b48f-29a642ac1f78"
+					(reference "U4")
+					(unit 1)
+				)
+				(path "/af2d881c-6553-449d-9093-6deb41497bdc/67eb63b8-4985-495d-ab9e-4c58fb498c7d"
+					(reference "U3")
+					(unit 1)
+				)
+				(path "/af2d881c-6553-449d-9093-6deb41497bdc/777ce27f-f0db-4b38-a663-f213b2d41686"
 					(reference "U1")
 					(unit 1)
 				)
-				(path "/af2d881c-6553-449d-9093-6deb41497bdc/67eb63b8-4985-495d-ab9e-4c58fb498c7d"
-					(reference "U5")
-					(unit 1)
-				)
-				(path "/af2d881c-6553-449d-9093-6deb41497bdc/777ce27f-f0db-4b38-a663-f213b2d41686"
+				(path "/af2d881c-6553-449d-9093-6deb41497bdc/97e743ff-8a82-4285-b0f3-f0e89ab922fa"
 					(reference "U2")
-					(unit 1)
-				)
-				(path "/af2d881c-6553-449d-9093-6deb41497bdc/97e743ff-8a82-4285-b0f3-f0e89ab922fa"
-					(reference "U3")
 					(unit 1)
 				)
@@
 		(on_board yes)
 		(dnp no)
-		(property "Reference" "R7"
-			(at 99.314 47.244 90)
+		(property "Reference" "R24"
+			(at 98.298 48.26 90)
 			(effects
 				(font
@@
 		)
 		(property "Value" "33"
-			(at 103.124 47.244 90)
+			(at 104.648 48.26 90)
 			(effects
 				(font
@@
 			(project "HackerDAQ Digital IO Card"
 				(path "/af2d881c-6553-449d-9093-6deb41497bdc/455d3721-42aa-4f0e-b48f-29a642ac1f78"
-					(reference "R3")
+					(reference "R19")
 					(unit 1)
 				)
 				(path "/af2d881c-6553-449d-9093-6deb41497bdc/67eb63b8-4985-495d-ab9e-4c58fb498c7d"
-					(reference "R15")
+					(reference "R31")
 					(unit 1)
 				)
 				(path "/af2d881c-6553-449d-9093-6deb41497bdc/777ce27f-f0db-4b38-a663-f213b2d41686"
-					(reference "R7")
+					(reference "R24")
 					(unit 1)
 				)
 				(path "/af2d881c-6553-449d-9093-6deb41497bdc/97e743ff-8a82-4285-b0f3-f0e89ab922fa"
-					(reference "R11")
-					(unit 1)
-				)
+					(reference "R27")
+					(unit 1)
+				)
