File: hardware/Digital IO Card/IOProtection.kicad_sch (KiCad schematic)
At the start: 5 parts, among them U1 SRV05-4.TCT

Commit message: Fix DRC/ERC errors
Parts:
- renumbered R5 to R10, R14 to R13, R24 to R25, R25 to R26, U1 to U2
Changed lines of the file:
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@@
 		(on_board yes)
 		(dnp no)
-		(property "Reference" "R14"
+		(property "Reference" "R13"
 			(at 93.726 48.006 90)
 			(effects
@@
 			(project "HackerDAQ Digital IO Card"
 				(path "/af2d881c-6553-449d-9093-6deb41497bdc/455d3721-42aa-4f0e-b48f-29a642ac1f78"
+					(reference "R16")
+					(unit 1)
+				)
+				(path "/af2d881c-6553-449d-9093-6deb41497bdc/67eb63b8-4985-495d-ab9e-4c58fb498c7d"
+					(reference "R15")
+					(unit 1)
+				)
+				(path "/af2d881c-6553-449d-9093-6deb41497bdc/777ce27f-f0db-4b38-a663-f213b2d41686"
 					(reference "R13")
 					(unit 1)
 				)
-				(path "/af2d881c-6553-449d-9093-6deb41497bdc/67eb63b8-4985-495d-ab9e-4c58fb498c7d"
-					(reference "R18")
-					(unit 1)
-				)
-				(path "/af2d881c-6553-449d-9093-6deb41497bdc/777ce27f-f0db-4b38-a663-f213b2d41686"
+				(path "/af2d881c-6553-449d-9093-6deb41497bdc/97e743ff-8a82-4285-b0f3-f0e89ab922fa"
 					(reference "R14")
-					(unit 1)
-				)
-				(path "/af2d881c-6553-449d-9093-6deb41497bdc/97e743ff-8a82-4285-b0f3-f0e89ab922fa"
-					(reference "R17")
 					(unit 1)
 				)
@@
 		(on_board yes)
 		(dnp no)
-		(property "Reference" "R25"
+		(property "Reference" "R26"
 			(at 102.616 55.626 90)
 			(effects
@@
 			(project "HackerDAQ Digital IO Card"
 				(path "/af2d881c-6553-449d-9093-6deb41497bdc/455d3721-42aa-4f0e-b48f-29a642ac1f78"
-					(reference "R20")
+					(reference "R32")
 					(unit 1)
 				)
 				(path "/af2d881c-6553-449d-9093-6deb41497bdc/67eb63b8-4985-495d-ab9e-4c58fb498c7d"
-					(reference "R32")
+					(reference "R30")
 					(unit 1)
 				)
 				(path "/af2d881c-6553-449d-9093-6deb41497bdc/777ce27f-f0db-4b38-a663-f213b2d41686"
-					(reference "R25")
+					(reference "R26")
 					(unit 1)
 				)
 				(path "/af2d881c-6553-449d-9093-6deb41497bdc/97e743ff-8a82-4285-b0f3-f0e89ab922fa"
-					(reference "R26")
+					(reference "R28")
 					(unit 1)
 				)
@@
 		(on_board yes)
 		(dnp no)
-		(property "Reference" "R5"
+		(property "Reference" "R10"
 			(at 89.154 40.386 90)
 			(effects
@@
 			(project "HackerDAQ Digital IO Card"
 				(path "/af2d881c-6553-449d-9093-6deb41497bdc/455d3721-42aa-4f0e-b48f-29a642ac1f78"
-					(reference "R1")
+					(reference "R6")
 					(unit 1)
 				)
@@
 				)
 				(path "/af2d881c-6553-449d-9093-6deb41497bdc/777ce27f-f0db-4b38-a663-f213b2d41686"
-					(reference "R5")
+					(reference "R10")
 					(unit 1)
 				)
 				(path "/af2d881c-6553-449d-9093-6deb41497bdc/97e743ff-8a82-4285-b0f3-f0e89ab922fa"
-					(reference "R8")
+					(reference "R11")
 					(unit 1)
 				)
@@
 		(dnp no)
 		(fields_autoplaced yes)
-		(property "Reference" "U1"
+		(property "Reference" "U2"
 			(at 69.1581 63.5 0)
 			(effects
@@
 			(project "HackerDAQ Digital IO Card"
 				(path "/af2d881c-6553-449d-9093-6deb41497bdc/455d3721-42aa-4f0e-b48f-29a642ac1f78"
-					(reference "U9")
+					(reference "U1")
 					(unit 1)
 				)
 				(path "/af2d881c-6553-449d-9093-6deb41497bdc/67eb63b8-4985-495d-ab9e-4c58fb498c7d"
+					(reference "U4")
+					(unit 1)
+				)
+				(path "/af2d881c-6553-449d-9093-6deb41497bdc/777ce27f-f0db-4b38-a663-f213b2d41686"
+					(reference "U2")
+					(unit 1)
+				)
+				(path "/af2d881c-6553-449d-9093-6deb41497bdc/97e743ff-8a82-4285-b0f3-f0e89ab922fa"
 					(reference "U3")
-					(unit 1)
-				)
-				(path "/af2d881c-6553-449d-9093-6deb41497bdc/777ce27f-f0db-4b38-a663-f213b2d41686"
-					(reference "U1")
-					(unit 1)
-				)
-				(path "/af2d881c-6553-449d-9093-6deb41497bdc/97e743ff-8a82-4285-b0f3-f0e89ab922fa"
-					(reference "U2")
 					(unit 1)
 				)
@@
 		(on_board yes)
 		(dnp no)
-		(property "Reference" "R24"
+		(property "Reference" "R25"
 			(at 98.298 48.26 90)
 			(effects
@@
 			(project "HackerDAQ Digital IO Card"
 				(path "/af2d881c-6553-449d-9093-6deb41497bdc/455d3721-42aa-4f0e-b48f-29a642ac1f78"
-					(reference "R19")
+					(reference "R31")
 					(unit 1)
 				)
 				(path "/af2d881c-6553-449d-9093-6deb41497bdc/67eb63b8-4985-495d-ab9e-4c58fb498c7d"
-					(reference "R31")
+					(reference "R29")
 					(unit 1)
 				)
 				(path "/af2d881c-6553-449d-9093-6deb41497bdc/777ce27f-f0db-4b38-a663-f213b2d41686"
-					(reference "R24")
-					(unit 1)
-				)
+					(reference "R25")
+					(unit 1)
+				)
