File: hardware/Digital IO Card/LEDDriver.kicad_sch (KiCad schematic)
At the start: 2 parts, among them U8 SN74ACT17PWR

Commit message: Finish redesigned DIO card
Parts:
- renumbered U8 to U5
Changed lines of the file:
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@@
 		(dnp no)
 		(fields_autoplaced yes)
-		(property "Reference" "U8"
+		(property "Reference" "U5"
 			(at 62.23 36.83 0)
 			(effects
@@
 			(project "HackerDAQ Digital IO Card"
 				(path "/af2d881c-6553-449d-9093-6deb41497bdc/367befd8-87f7-4a27-a26f-a85b1cb947a6"
-					(reference "U8")
+					(reference "U5")
 					(unit 1)
 				)
 				(path "/af2d881c-6553-449d-9093-6deb41497bdc/74ac3964-50d1-4760-8013-20b90da47d63"
+					(reference "U7")
+					(unit 1)
+				)
+				(path "/af2d881c-6553-449d-9093-6deb41497bdc/86043100-9ecf-4922-ba85-a69132f1d586"
 					(reference "U6")
 					(unit 1)
 				)
-				(path "/af2d881c-6553-449d-9093-6deb41497bdc/86043100-9ecf-4922-ba85-a69132f1d586"
-					(reference "U9")
-					(unit 1)
-				)
