File: hardware/Digital IO Card/LEDDriver.kicad_sch (KiCad schematic)
At the start: 2 parts, among them U5 SN74ACT17PWR

Commit message: Fix DRC/ERC errors
Parts:
- renumbered C2 to C1
Changed lines of the file:
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@@
 				)
 				(path "/af2d881c-6553-449d-9093-6deb41497bdc/74ac3964-50d1-4760-8013-20b90da47d63"
-					(reference "U7")
+					(reference "U6")
 					(unit 1)
 				)
 				(path "/af2d881c-6553-449d-9093-6deb41497bdc/86043100-9ecf-4922-ba85-a69132f1d586"
-					(reference "U6")
+					(reference "U7")
 					(unit 1)
 				)
@@
 		(on_board yes)
 		(dnp no)
-		(property "Reference" "C2"
+		(property "Reference" "C1"
 			(at 38.1 35.5662 0)
 			(effects
@@
 			(project "HackerDAQ Digital IO Card"
 				(path "/af2d881c-6553-449d-9093-6deb41497bdc/367befd8-87f7-4a27-a26f-a85b1cb947a6"
+					(reference "C1")
+					(unit 1)
+				)
+				(path "/af2d881c-6553-449d-9093-6deb41497bdc/74ac3964-50d1-4760-8013-20b90da47d63"
 					(reference "C2")
 					(unit 1)
 				)
-				(path "/af2d881c-6553-449d-9093-6deb41497bdc/74ac3964-50d1-4760-8013-20b90da47d63"
-					(reference "C1")
-					(unit 1)
-				)
