File: hardware/Digital IO Card/LevelShifter.kicad_sch (KiCad schematic)
At the start: 9 parts, among them U10 TXB0106PW, U11 SN74AHC1G125

Commit message: Back-annotate
Parts:
- renumbered D3 to D4
Changed lines of the file:
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@@
 		(on_board yes)
 		(dnp no)
-		(property "Reference" "D3"
+		(property "Reference" "D4"
 			(at 90.17 138.1126 90)
 			(effects
@@
 			(project "HackerDAQ Digital IO Card"
 				(path "/af2d881c-6553-449d-9093-6deb41497bdc/5489c672-23f8-4c65-8a7e-45865ecb61e5"
-					(reference "D3")
+					(reference "D4")
 					(unit 1)
 				)
