File: hardware/Digital IO Card/LevelShifter.kicad_sch (KiCad schematic)
At the start: 9 parts, among them U10 TXB0106PW, U11 SN74AHC1G125

Commit message: Fix DRC/ERC errors
Parts:
- renumbered U11 to U10, U10 to U11

Commit message: Designator conflict :(
Changed lines of the file:
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@@
+	)
+	(bus_entry
+		(at 223.52 62.23)
+		(size -2.54 2.54)
+		(stroke
+			(width 0)
+			(type default)
+		)
 	)
 	(bus_entry
@@
 	)
 	(bus_entry
+		(at 223.52 58.42)
+		(size -2.54 2.54)
+		(stroke
+			(width 0)
+			(type default)
+		)
+	)
+	(bus_entry
 		(at 227.33 54.61)
 		(size -2.54 2.54)
@@
 	)
 	(bus_entry
-		(at 227.33 57.15)
+		(at 227.33 52.07)
 		(size -2.54 2.54)
 		(stroke
@@
 	)
 	(bus_entry
-		(at 223.52 49.53)
+		(at 121.92 125.73)
+		(size 2.54 2.54)
+		(stroke
+			(width 0)
+			(type default)
+		)
+	)
+	(bus_entry
+		(at 121.92 62.23)
+		(size 2.54 2.54)
+		(stroke
+			(width 0)
+			(type default)
+		)
+	)
+	(bus_entry
+		(at 113.03 123.19)
+		(size 2.54 2.54)
+		(stroke
+			(width 0)
+			(type default)
+		)
+	)
+	(bus_entry
+		(at 116.84 54.61)
+		(size 2.54 2.54)
+		(stroke
+			(width 0)
+			(type default)
+		)
+	)
+	(bus_entry
+		(at 101.6 123.19)
+		(size 2.54 2.54)
+		(stroke
+			(width 0)
+			(type default)
+		)
+	)
+	(bus_entry
+		(at 227.33 49.53)
 		(size -2.54 2.54)
 		(stroke
@@
 	)
 	(bus_entry
-		(at 121.92 125.73)
-		(size 2.54 2.54)
-		(stroke
-			(width 0)
-			(type default)
-		)
-	)
-	(bus_entry
-		(at 121.92 62.23)
-		(size 2.54 2.54)
-		(stroke
-			(width 0)
-			(type default)
-		)
-	)
-	(bus_entry
-		(at 113.03 123.19)
-		(size 2.54 2.54)
-		(stroke
-			(width 0)
-			(type default)
-		)
-	)
-	(bus_entry
-		(at 227.33 62.23)
-		(size -2.54 2.54)
-		(stroke
-			(width 0)
-			(type default)
-		)
-	)
-	(bus_entry
-		(at 116.84 54.61)
-		(size 2.54 2.54)
-		(stroke
-			(width 0)
-			(type default)
-		)
-	)
-	(bus_entry
-		(at 223.52 52.07)
-		(size -2.54 2.54)
-		(stroke
-			(width 0)
-			(type default)
-		)
-	)
-	(bus_entry
-		(at 101.6 123.19)
-		(size 2.54 2.54)
-		(stroke
-			(width 0)
-			(type default)
-		)
-	)
-	(bus_entry
 		(at 90.17 123.19)
 		(size 2.54 2.54)
@@
 	(wire
 		(pts
-			(xy 181.61 64.77) (xy 224.79 64.77)
+			(xy 181.61 64.77) (xy 220.98 64.77)
 		)
 		(stroke
@@
 		)
 	)
+	(bus
+		(pts
+			(xy 227.33 49.53) (xy 227.33 52.07)
+		)
+		(stroke
+			(width 0)
+			(type default)
+		)
+	)
 	(wire
 		(pts
@@
 		)
 	)
+	(wire
+		(pts
+			(xy 220.98 60.96) (xy 219.71 60.96)
+		)
+		(stroke
+			(width 0)
+			(type default)
+		)
+	)
 	(bus
 		(pts
@@
 		)
 	)
+	(bus
+		(pts
+			(xy 227.33 52.07) (xy 227.33 54.61)
+		)
+		(stroke
+			(width 0)
+			(type default)
+		)
+	)
 	(wire
 		(pts
@@
 		)
 	)
-	(bus
-		(pts
-			(xy 223.52 52.07) (xy 223.52 125.73)
-		)
-		(stroke
-			(width 0)
-			(type default)
-		)
-	)
 	(wire
 		(pts
@@
 	(wire
 		(pts
-			(xy 181.61 52.07) (xy 220.98 52.07)
+			(xy 181.61 52.07) (xy 224.79 52.07)
 		)
 		(stroke
@@
 	(bus
 		(pts
-			(xy 223.52 49.53) (xy 223.52 52.07)
-		)
-		(stroke
-			(width 0)
-			(type default)
-		)
-	)
-	(bus
-		(pts
 			(xy 229.87 41.91) (xy 223.52 41.91)
 		)
@@
 	(bus
 		(pts
-			(xy 227.33 54.61) (xy 227.33 57.15)
+			(xy 223.52 62.23) (xy 223.52 125.73)
 		)
 		(stroke
@@
 	(bus
 		(pts
-			(xy 227.33 57.15) (xy 227.33 62.23)
-		)
-		(stroke
-			(width 0)
-			(type default)
-		)
-	)
-	(bus
-		(pts
 			(xy 121.92 62.23) (xy 121.92 125.73)
 		)
@@
 	(bus
 		(pts
-			(xy 227.33 62.23) (xy 227.33 88.9)
+			(xy 223.52 58.42) (xy 223.52 62.23)
+		)
+		(stroke
+			(width 0)
+			(type default)
+		)
+	)
+	(bus
+		(pts
+			(xy 227.33 54.61) (xy 227.33 88.9)
 		)
 		(stroke
@@
 	(bus
 		(pts
-			(xy 227.33 44.45) (xy 227.33 54.61)
+			(xy 227.33 44.45) (xy 227.33 49.53)
 		)
 		(stroke
@@
 		)
 	)
+	(wire
+		(pts
+			(xy 219.71 60.96) (xy 219.71 59.69)
+		)
+		(stroke
+			(width 0)
+			(type default)
+		)
+	)
 	(bus
 		(pts
@@
 	(bus
 		(pts
-			(xy 223.52 41.91) (xy 223.52 49.53)
+			(xy 223.52 41.91) (xy 223.52 58.42)
 		)
 		(stroke
@@
 	(wire
 		(pts
-			(xy 181.61 59.69) (xy 224.79 59.69)
-		)
-		(stroke
-			(width 0)
-			(type default)
-		)
-	)
-	(wire
-		(pts
-			(xy 181.61 54.61) (xy 220.98 54.61)
-		)
-		(stroke
+			(xy 181.61 59.69) (xy 219.71 59.69)
+		)
+		(stroke
+			(width 0)
+			(type default)
+		)
+	)
+	(wire
+		(pts
+			(xy 181.61 54.61) (xy 224.79 54.61)
+		)
+		(stroke
