File: hardware/High Current Output Card/IOExpander.kicad_sch (KiCad schematic)
At the start: 2 parts, among them U8 MCP23S17_SS

Commit message: Finish redesigned DIO card
Parts:
- renumbered C4 to C51, U8 to U34
Connections:
- net PA0: no longer names the net of U34.21 (GPA0)
- net PA1: no longer names the net of U34.22 (GPA1)
- net PA2 renamed DIG_IN3
- net PA3 renamed PULL_LOGIC_CTRL3
- net PA4 renamed HICUR_LOGIC_CTRL3
- net PA5 renamed DIG_IN2
- net PA6 renamed PULL_LOGIC_CTRL2
- net PA7 renamed HICUR_LOGIC_CTRL2
- net PB0 renamed DIG_IN1
- net PB1 renamed PULL_LOGIC_CTRL1
- net PB2 renamed HICUR_LOGIC_CTRL1
- net PB3 renamed DIG_IN0
- net PB4 renamed PULL_LOGIC_CTRL0
- net PB5 renamed HICUR_LOGIC_CTRL0
- net PB6: no longer names the net of U34.7 (GPB6)
- net PB7: no longer names the net of U34.8 (GPB7)
- net SPI.MISO renamed SPI_5V.MISO
- net SPI.MOSI renamed SPI_5V.MOSI
- net SPI.SCLK renamed SPI_5V.SCLK
- net V_{DD} renamed +5V
- no-connect marks 2 -> 6
Other:
- note added: "This circuit implements enough I/O for one bank of digital front ends via an MCP23S17 16-bit I/O expander. This allows them to be controlled using SPI commands at a clock of up to 10MHz. Note that the expander is powered off of 5V in order to produce 5V I/O for the front ends."
- note removed: "This circuit implements enough I/O for one bank of digital front ends via an MCP23S17 16-bit I/O expander. This allows them to be controlled using SPI commands at a clock of up to 10MHz. Note that the expander may be powered off of 1.8-5.5V."
- moved on the sheet: C51, U34
