File: hardware/High Current Output Card/LevelShifter.kicad_sch (KiCad schematic)
At the start: 9 parts, among them U10 TXB0106PW, U11 SN74AHC1G125

Commit message: Finish redesigned DIO card
Parts:
- removed C7: 100nF, Capacitor_SMD:C_0603_1608Metric, symbol Device:C_Small
- removed U10: TXB0106PW, Package_SO:TSSOP-16_4.4x5mm_P0.65mm, symbol Logic_LevelTranslator:TXB0106PW
- added U36: SN74ACT17PWR, Package_SO:TSSOP-14_4.4x5mm_P0.65mm, symbol Project Library:SN74ACT17
- renumbered C6 to C52, D2 to D10, D3 to D11, D1 to D9, R35 to R106, R34 to R107, U11 to U38
Connections:
- net GND: now also U36.7 (GND)
- net SPI.MOSI: now also U36.1 (1A)
- net SPI.SCLK: now also U36.3 (2A)
- net ~{CS}0: now also U36.5 (3A)
- net ~{CS}1: now also U36.9 (4A)
- net ~{CS}2: now also U36.11 (5A)
- net ~{RESET}: now also U36.13 (6A)
- net SPI_VL.MISO renamed SPI_5V.MISO
- net V_{LOGIC} renamed +5V
- net +5V: now also U36.14 (V_{CC})
- new net SPI_5V.MOSI: U36.2 (1Y)
- new net SPI_5V.SCLK: U36.4 (2Y)
- new net ~{CS_5V}0: U36.6 (3Y)
- new net ~{CS_5V}1: U36.8 (4Y)
- new net ~{CS_5V}2: U36.10 (5Y)
- new net ~{RESET_5V}: U36.12 (6Y)
Other:
- moved on the sheet: C52
