File: hardware/Main Unit/Main Unit.kicad_pcb (KiCad board)
At the start: 4 copper layers, 147 parts, among them J1 3221-10-0300-00, J10 DM3AT, J11 USB4105-GF-A, J13 HFJ11-2450E-L21RL, J2 61801525123, J3 61801525123, J4 61801525123, J5 61801525123, J6 61801525123, J7 61801525123, J8 61801525123, J9 61801525123, SW1 MJTP1243, SW2 MJTP1243, U1 MCXN547VKLT, U10 USBLC6-2SC6, U11 TPS56A37RPAR, U12 INA180A3, U2 CY7C65223, U2 TLV71333PDBV, U3 SN74CB3Q3257PWR, U4 SN74CB3Q3257PWR, U5 SN74CB3Q3257PWR, U6 SN74CB3Q3257PWR, U7 74AHC1G04, U7 KSZ8081RND, U8 AP22913W6-7, U9 SN74AXC4T774, X1 24.0000MHz

Commit message: Main unit: Add USB port for MCU and 3.3VA rail, start on routing
Parts:
- removed the C1 at (153.7, 114.9)
- removed the C2 at (153.7, 117.5)
- removed the C30 at (183.8, 93.3)
- removed the C32 at (183.8, 96.6)
- removed the R12 at (191.4, 79.5)
- removed the R13 at (191.4, 82.9)
- removed the R14 at (191.4, 86.2)
- removed the R16 at (191.4, 89.5)
- removed the R17 at (191.4, 92.8)
- removed TP5: +3.3VA, TestPoint:TestPoint_THTPad_D2.5mm_Drill1.2mm
- removed the U2 at (158.2, 116.1)
- removed the U7 at (196.8, 70.4)
- added C52: 100nF, Capacitor_SMD:C_0603_1608Metric, F.Cu at (146.9, 109.0)
- added C53: 100nF, Capacitor_SMD:C_0603_1608Metric, F.Cu at (102.8, 62.5)
- added C54: 1µF, Capacitor_SMD:C_0603_1608Metric, F.Cu at (102.8, 59.5)
- added J12: USB4105-GF-A, Project Library:USB_C_Receptacle_GCT_USB4105-xx-A_16P_TopMnt_Horizontal-ExtraHoleClearance, F.Cu at (125.0, 40.8)
- added R41: 5.1k, Resistor_SMD:R_0603_1608Metric, F.Cu at (120.1, 47.7)
- added R42: 5.1k, Resistor_SMD:R_0603_1608Metric, F.Cu at (120.1, 50.2)
- added U13: USBLC6-2SC6, Package_TO_SOT_SMD:SOT-23-6, F.Cu at (115.5, 48.9)
- added U14: CY7C65223, Project Library:QFN-24-1EP_4x4mm_P0.5mm_EP2.65x2.65mm-LengthenedPads, F.Cu at (108.0, 63.3)
- added X2: 8.192MHz, Oscillator:Oscillator_SMD_ECS_2520MV-xxx-xx-4Pin_2.5x2.0mm, F.Cu at (146.8, 112.4)
- C1: value 1µF -> 100nF
- C2: value 100nF -> 1µF
- R10, R11, R2, R3, R4: footprint Resistor_SMD:R_1206_3216Metric -> Resistor_SMD:R_0603_1608Metric
- R15: value 10k -> 5.1k; footprint Resistor_SMD:R_1206_3216Metric -> Resistor_SMD:R_0603_1608Metric
- U2: value CY7C65223 -> TLV71333PDBV; footprint Project Library:QFN-24-1EP_4x4mm_P0.5mm_EP2.65x2.65mm-LengthenedPads -> Package_TO_SOT_SMD:SOT-23-5
- moved C20 234.8 mm to (342.8, 296.2)
- moved R1 234.8 mm to (342.8, 301.2)
- moved C14 234.8 mm to (340.2, 279.7)
- moved C24 234.8 mm to (335.4, 286.9)
- moved R18 234.8 mm to (307.4, 287.9)
- moved SW1 234.8 mm to (332.4, 295.0)
- moved SW2 234.8 mm to (332.4, 300.0)
- moved TP1 234.8 mm to (339.7, 290.4)
- moved C19 234.8 mm to (342.8, 293.7)
- moved D1 234.8 mm to (332.7, 304.6)
- moved R2 234.8 mm to (337.7, 304.2)
- moved D5 211.4 mm to (32.2, 6.75)
- moved R37 211.4 mm to (33.1, 3.76)
- moved C43 190.3 mm to (59.2, 47.2)
- moved C44 190.3 mm to (55.8, 47.2)
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Connections:
- net /MCU/uSD_SPI_FC6.MISO renamed /uSD_SPI.MISO
- net /MCU/uSD_SPI_FC6.MOSI renamed /uSD_SPI.MOSI
- net /MCU/uSD_SPI_FC6.SCLK renamed /uSD_SPI.SCLK
- net /MCU/uSD_SPI_FC6.~{CS} renamed /uSD_SPI.~{CS}
- net /MCU/~{SD_CARD_EN} renamed /~{SD_CARD_EN}
- C1 pad 1: /DebugUSBUART/USBSER_VCCD -> +5V
- C10 pad 1: +3.3V -> +3.3VA
- C11 pad 1: +3.3V -> +3.3VA
- C19 pad 1: /EthernetInterface/~{RST} -> /~{MCU_RST}
- C2 pad 1: +3.3V -> +3.3VA
- D1 pad 1: /EthernetInterface/~{RST} -> /~{MCU_RST}
- J1 pad 10: /EthernetInterface/~{RST} -> /~{MCU_RST}
- J2 pad 10: /CARD_BUS_0_SPI.~{DRDY} -> /CARD_BUS_1_SPI.~{DRDY}
- J2 pad 12: /CARD_BUS_0_SPI.MISO -> /CARD_BUS_1_SPI.MISO
- J2 pad 13: /CARD_BUS_0_SPI.MOSI -> /CARD_BUS_1_SPI.MOSI
- J2 pad 14: /CARD_BUS_0_SPI.SCLK -> /CARD_BUS_1_SPI.SCLK
- J2 pad 15: /Card Bus Connectors0/CARD_CS.~{CS}1 -> /Card Bus Connectors1/L_CARD_CS.~{CS}1
- J2 pad 4: /Card Bus Connectors0/8.192MHZ_CLK -> /8.192MHZ_CLK
- J2 pad 7: /Card Bus Connectors0/CARD_CS.~{CS}2 -> /Card Bus Connectors1/L_CARD_CS.~{CS}2
- J2 pad 8: /Card Bus Connectors0/CARD_CS.~{CS}0 -> /Card Bus Connectors1/L_CARD_CS.~{CS}0
- J3 pad 10: /CARD_BUS_0_SPI.~{DRDY} -> /CARD_BUS_1_SPI.~{DRDY}
- J3 pad 12: /CARD_BUS_0_SPI.MISO -> /CARD_BUS_1_SPI.MISO
- J3 pad 13: /CARD_BUS_0_SPI.MOSI -> /CARD_BUS_1_SPI.MOSI
- J3 pad 14: /CARD_BUS_0_SPI.SCLK -> /CARD_BUS_1_SPI.SCLK
- J3 pad 15: /Card Bus Connectors0/CARD_CS.~{CS}1 -> /Card Bus Connectors1/F_CARD_CS.~{CS}1
- J3 pad 4: /Card Bus Connectors0/8.192MHZ_CLK -> /8.192MHZ_CLK
- J3 pad 7: /Card Bus Connectors0/CARD_CS.~{CS}2 -> /Card Bus Connectors1/F_CARD_CS.~{CS}2
- J3 pad 8: /Card Bus Connectors0/CARD_CS.~{CS}0 -> /Card Bus Connectors1/F_CARD_CS.~{CS}0
- J4 pad 10: /CARD_BUS_1_SPI.~{DRDY} -> /CARD_BUS_0_SPI.~{DRDY}
- J4 pad 11: /Card Bus Connectors1/~{SYNC} -> /Card Bus Connectors0/~{SYNC}
- J4 pad 12: /CARD_BUS_1_SPI.MISO -> /CARD_BUS_0_SPI.MISO
- J4 pad 13: /CARD_BUS_1_SPI.MOSI -> /CARD_BUS_0_SPI.MOSI
- J4 pad 14: /CARD_BUS_1_SPI.SCLK -> /CARD_BUS_0_SPI.SCLK
- J4 pad 15: /Card Bus Connectors1/CARD_CS.~{CS}1 -> /Card Bus Connectors0/L_CARD_CS.~{CS}1
- J4 pad 4: /Card Bus Connectors1/8.192MHZ_CLK -> /8.192MHZ_CLK
- J4 pad 6: /Card Bus Connectors1/~{RESET} -> /Card Bus Connectors0/~{RESET}
- J4 pad 7: /Card Bus Connectors1/CARD_CS.~{CS}2 -> /Card Bus Connectors0/L_CARD_CS.~{CS}2
- J4 pad 8: /Card Bus Connectors1/CARD_CS.~{CS}0 -> /Card Bus Connectors0/L_CARD_CS.~{CS}0
- J5 pad 10: /CARD_BUS_1_SPI.~{DRDY} -> /CARD_BUS_0_SPI.~{DRDY}
- J5 pad 11: /Card Bus Connectors1/~{SYNC} -> /Card Bus Connectors0/~{SYNC}
- J5 pad 12: /CARD_BUS_1_SPI.MISO -> /CARD_BUS_0_SPI.MISO
- J5 pad 13: /CARD_BUS_1_SPI.MOSI -> /CARD_BUS_0_SPI.MOSI
- J5 pad 14: /CARD_BUS_1_SPI.SCLK -> /CARD_BUS_0_SPI.SCLK
- J5 pad 15: /Card Bus Connectors1/CARD_CS.~{CS}1 -> /Card Bus Connectors0/F_CARD_CS.~{CS}1
- J5 pad 4: /Card Bus Connectors1/8.192MHZ_CLK -> /8.192MHZ_CLK
- J5 pad 6: /Card Bus Connectors1/~{RESET} -> /Card Bus Connectors0/~{RESET}
- J5 pad 7: /Card Bus Connectors1/CARD_CS.~{CS}2 -> /Card Bus Connectors0/F_CARD_CS.~{CS}2
- J5 pad 8: /Card Bus Connectors1/CARD_CS.~{CS}0 -> /Card Bus Connectors0/F_CARD_CS.~{CS}0
- J6 pad 11: /Card Bus Connectors2/~{SYNC} -> /Card Bus Connectors0/~{SYNC}
- J6 pad 15: /Card Bus Connectors2/CARD_CS.~{CS}1 -> /Card Bus Connectors2/L_CARD_CS.~{CS}1
- J6 pad 4: /Card Bus Connectors2/8.192MHZ_CLK -> /8.192MHZ_CLK
- J6 pad 6: /Card Bus Connectors2/~{RESET} -> /Card Bus Connectors0/~{RESET}
- J6 pad 7: /Card Bus Connectors2/CARD_CS.~{CS}2 -> /Card Bus Connectors2/L_CARD_CS.~{CS}2
- J6 pad 8: /Card Bus Connectors2/CARD_CS.~{CS}0 -> /Card Bus Connectors2/L_CARD_CS.~{CS}0
- J7 pad 11: /Card Bus Connectors2/~{SYNC} -> /Card Bus Connectors0/~{SYNC}
- J7 pad 15: /Card Bus Connectors2/CARD_CS.~{CS}1 -> /Card Bus Connectors2/F_CARD_CS.~{CS}1
- J7 pad 4: /Card Bus Connectors2/8.192MHZ_CLK -> /8.192MHZ_CLK
- J7 pad 6: /Card Bus Connectors2/~{RESET} -> /Card Bus Connectors0/~{RESET}
- J7 pad 7: /Card Bus Connectors2/CARD_CS.~{CS}2 -> /Card Bus Connectors2/F_CARD_CS.~{CS}2
- J7 pad 8: /Card Bus Connectors2/CARD_CS.~{CS}0 -> /Card Bus Connectors2/F_CARD_CS.~{CS}0
- J8 pad 11: /Card Bus Connectors3/~{SYNC} -> /Card Bus Connectors0/~{SYNC}
- J8 pad 15: /Card Bus Connectors3/CARD_CS.~{CS}1 -> /Card Bus Connectors3/L_CARD_CS.~{CS}1
- J8 pad 4: /Card Bus Connectors3/8.192MHZ_CLK -> /8.192MHZ_CLK
- J8 pad 6: /Card Bus Connectors3/~{RESET} -> /Card Bus Connectors0/~{RESET}
- J8 pad 7: /Card Bus Connectors3/CARD_CS.~{CS}2 -> /Card Bus Connectors3/L_CARD_CS.~{CS}2
- J8 pad 8: /Card Bus Connectors3/CARD_CS.~{CS}0 -> /Card Bus Connectors3/L_CARD_CS.~{CS}0
- J9 pad 11: /Card Bus Connectors3/~{SYNC} -> /Card Bus Connectors0/~{SYNC}
- J9 pad 15: /Card Bus Connectors3/CARD_CS.~{CS}1 -> /Card Bus Connectors3/F_CARD_CS.~{CS}1
- J9 pad 4: /Card Bus Connectors3/8.192MHZ_CLK -> /8.192MHZ_CLK
- J9 pad 6: /Card Bus Connectors3/~{RESET} -> /Card Bus Connectors0/~{RESET}
- J9 pad 7: /Card Bus Connectors3/CARD_CS.~{CS}2 -> /Card Bus Connectors3/F_CARD_CS.~{CS}2
- J9 pad 8: /Card Bus Connectors3/CARD_CS.~{CS}0 -> /Card Bus Connectors3/F_CARD_CS.~{CS}0
- R1 pad 1: /EthernetInterface/~{RST} -> /~{MCU_RST}
- R10 pad 1: /MicroSDCard/DET_B -> GND
- R10 pad 2: GND -> /MicroSDCard/DET_B
- R11 pad 1: /MicroSDCard/CLK@SD -> GND
- R11 pad 2: GND -> /MicroSDCard/CLK@SD
- R15 pad 1: /MCU/~{RST} -> GND
- R15 pad 2: +3.3V -> Net-(J11-CC1)
- R23 pad 1: /EthernetInterface/~{RST} -> /~{MCU_RST}
- R5 pad 1: /Card Bus Connectors0/CARD_CS.~{CS}0 -> unconnected-(R5-R1-Pad1)
- R5 pad 2: /Card Bus Connectors0/CARD_CS.~{CS}0 -> /Card Bus Connectors1/F_CARD_CS.~{CS}0
- R5 pad 3: /Card Bus Connectors0/CARD_CS.~{CS}1 -> /Card Bus Connectors1/F_CARD_CS.~{CS}1
- R5 pad 4: /Card Bus Connectors0/CARD_CS.~{CS}1 -> /Card Bus Connectors1/F_CARD_CS.~{CS}2
- R5 pad 6: /Card Bus Connectors0/CARD_CS.~{CS}2 -> /Card Bus Connectors1/L_CARD_CS.~{CS}2
- R5 pad 7: /Card Bus Connectors0/CARD_CS.~{CS}2 -> /Card Bus Connectors1/L_CARD_CS.~{CS}1
- R5 pad 8: unconnected-(R5-R7-Pad8) -> /Card Bus Connectors1/L_CARD_CS.~{CS}0
- R6 pad 1: /Card Bus Connectors1/CARD_CS.~{CS}0 -> unconnected-(R6-R1-Pad1)
- R6 pad 2: /Card Bus Connectors1/CARD_CS.~{CS}0 -> /Card Bus Connectors0/F_CARD_CS.~{CS}0
- R6 pad 3: /Card Bus Connectors1/CARD_CS.~{CS}1 -> /Card Bus Connectors0/F_CARD_CS.~{CS}1
- R6 pad 4: /Card Bus Connectors1/CARD_CS.~{CS}1 -> /Card Bus Connectors0/F_CARD_CS.~{CS}2
- R6 pad 6: /Card Bus Connectors1/CARD_CS.~{CS}2 -> /Card Bus Connectors0/L_CARD_CS.~{CS}2
- R6 pad 7: /Card Bus Connectors1/CARD_CS.~{CS}2 -> /Card Bus Connectors0/L_CARD_CS.~{CS}1
- R6 pad 8: unconnected-(R6-R7-Pad8) -> /Card Bus Connectors0/L_CARD_CS.~{CS}0
- R7 pad 1: /Card Bus Connectors2/CARD_CS.~{CS}0 -> unconnected-(R7-R1-Pad1)
- R7 pad 2: /Card Bus Connectors2/CARD_CS.~{CS}0 -> /Card Bus Connectors2/F_CARD_CS.~{CS}0
- R7 pad 3: /Card Bus Connectors2/CARD_CS.~{CS}1 -> /Card Bus Connectors2/F_CARD_CS.~{CS}1
- R7 pad 4: /Card Bus Connectors2/CARD_CS.~{CS}1 -> /Card Bus Connectors2/F_CARD_CS.~{CS}2
- R7 pad 6: /Card Bus Connectors2/CARD_CS.~{CS}2 -> /Card Bus Connectors2/L_CARD_CS.~{CS}2
- R7 pad 7: /Card Bus Connectors2/CARD_CS.~{CS}2 -> /Card Bus Connectors2/L_CARD_CS.~{CS}1
- R7 pad 8: unconnected-(R7-R7-Pad8) -> /Card Bus Connectors2/L_CARD_CS.~{CS}0
- R8 pad 1: /Card Bus Connectors3/CARD_CS.~{CS}0 -> unconnected-(R8-R1-Pad1)
- R8 pad 2: /Card Bus Connectors3/CARD_CS.~{CS}0 -> /Card Bus Connectors3/F_CARD_CS.~{CS}0
- R8 pad 3: /Card Bus Connectors3/CARD_CS.~{CS}1 -> /Card Bus Connectors3/F_CARD_CS.~{CS}1
- R8 pad 4: /Card Bus Connectors3/CARD_CS.~{CS}1 -> /Card Bus Connectors3/F_CARD_CS.~{CS}2
- R8 pad 6: /Card Bus Connectors3/CARD_CS.~{CS}2 -> /Card Bus Connectors3/L_CARD_CS.~{CS}2
- R8 pad 7: /Card Bus Connectors3/CARD_CS.~{CS}2 -> /Card Bus Connectors3/L_CARD_CS.~{CS}1
- R8 pad 8: unconnected-(R8-R7-Pad8) -> /Card Bus Connectors3/L_CARD_CS.~{CS}0
- SW1 pad 2: /EthernetInterface/~{RST} -> /~{MCU_RST}
- U1 pad 1: /CARD_BUS_0_SPI.MOSI -> /CARD_BUS_1_SPI.MOSI
- U1 pad 14: /CARD_BUS_3_SPI.~{CS}1 -> /CARD_BUS_0_SPI.~{CS}1
- U1 pad 15: /CARD_BUS_3_SPI.CARD_SEL -> /CARD_BUS_0_SPI.CARD_SEL
- U1 pad 16: /CARD_BUS_3_SPI.~{CS}0 -> /CARD_BUS_0_SPI.~{CS}0
- U1 pad 17: /CARD_BUS_3_SPI.SCLK -> /CARD_BUS_0_SPI.SCLK
- U1 pad 18: /CARD_BUS_3_SPI.MOSI -> /CARD_BUS_0_SPI.MOSI
- U1 pad 19: /CARD_BUS_3_SPI.MISO -> /CARD_BUS_0_SPI.MISO
- U1 pad 2: /CARD_BUS_0_SPI.SCLK -> /CARD_BUS_1_SPI.SCLK
- U1 pad 20: /CARD_BUS_3_SPI.~{DRDY} -> /CARD_BUS_0_SPI.~{DRDY}
- U1 pad 21: /CARD_BUS_3_SPI.~{CS}2 -> /CARD_BUS_0_SPI.~{CS}2
- U1 pad 27: unconnected-(U1E-P4_5-Pad27) -> /Card Bus Connectors0/~{RESET}
- U1 pad 28: unconnected-(U1E-P4_6-Pad28) -> /Card Bus Connectors0/~{SYNC}
- U1 pad 3: /CARD_BUS_0_SPI.MISO -> /CARD_BUS_1_SPI.MISO
- U1 pad 34: +3.3V -> +3.3VA
- U1 pad 4: /CARD_BUS_0_SPI.~{CS}0 -> /CARD_BUS_1_SPI.~{CS}0
- U1 pad 40: unconnected-(U1F-USB1_DP-Pad40) -> /MCU/USBMCU_D+
- U1 pad 41: unconnected-(U1F-USB1_DM-Pad41) -> /MCU/USBMCU_D-
- U1 pad 42: unconnected-(U1F-USB1_VBUS-Pad42) -> /MCU/USBMCU_VBUS
- U1 pad 50: /CARD_BUS_1_SPI.CARD_SEL -> /CARD_BUS_3_SPI.CARD_SEL
- U1 pad 51: /CARD_BUS_1_SPI.~{DRDY} -> /CARD_BUS_3_SPI.~{DRDY}
- U1 pad 65: /CARD_BUS_1_SPI.~{CS}0 -> /CARD_BUS_3_SPI.~{CS}0
- U1 pad 69: /CARD_BUS_1_SPI.MISO -> /CARD_BUS_3_SPI.MISO
- U1 pad 70: /CARD_BUS_1_SPI.MOSI -> /CARD_BUS_3_SPI.MOSI
- U1 pad 71: /CARD_BUS_1_SPI.SCLK -> /CARD_BUS_3_SPI.SCLK
- U1 pad 78: /CARD_BUS_1_SPI.~{CS}1 -> /CARD_BUS_3_SPI.~{CS}1
- U1 pad 79: /CARD_BUS_1_SPI.~{CS}2 -> /CARD_BUS_3_SPI.~{CS}2
- U1 pad 90: /CARD_BUS_0_SPI.~{CS}1 -> /CARD_BUS_1_SPI.~{CS}1
- U1 pad 91: /CARD_BUS_0_SPI.CARD_SEL -> /CARD_BUS_1_SPI.CARD_SEL
- U1 pad 92: /CARD_BUS_0_SPI.~{CS}2 -> /CARD_BUS_1_SPI.~{CS}2
- U1 pad 93: /CARD_BUS_0_SPI.~{DRDY} -> /CARD_BUS_1_SPI.~{DRDY}
- U11 pad 4: /EthernetInterface/~{RST} -> /~{MCU_RST}
- U2 pad 1: /DBG_UART.MCU_TX -> +5V
- U2 pad 2: unconnected-(U2-~{DTR}-Pad2) -> GND
- U2 pad 3: GND -> /~{MCU_RST}
- U2 pad 5: GND -> +3.3VA
- U3 pad 1: /CARD_BUS_0_SPI.CARD_SEL -> /CARD_BUS_1_SPI.CARD_SEL
- U3 pad 10: /Card Bus Connectors0/CARD_CS.~{CS}2 -> /Card Bus Connectors1/F_CARD_CS.~{CS}2
- U3 pad 11: /Card Bus Connectors0/CARD_CS.~{CS}2 -> /Card Bus Connectors1/L_CARD_CS.~{CS}2
- U3 pad 2: /Card Bus Connectors0/CARD_CS.~{CS}0 -> /Card Bus Connectors1/L_CARD_CS.~{CS}0
- U3 pad 3: /Card Bus Connectors0/CARD_CS.~{CS}0 -> /Card Bus Connectors1/F_CARD_CS.~{CS}0
- U3 pad 4: /CARD_BUS_0_SPI.~{CS}0 -> /CARD_BUS_1_SPI.~{CS}0
- U3 pad 5: /Card Bus Connectors0/CARD_CS.~{CS}1 -> /Card Bus Connectors1/L_CARD_CS.~{CS}1
- U3 pad 6: /Card Bus Connectors0/CARD_CS.~{CS}1 -> /Card Bus Connectors1/F_CARD_CS.~{CS}1
- U3 pad 7: /CARD_BUS_0_SPI.~{CS}1 -> /CARD_BUS_1_SPI.~{CS}1
- U3 pad 9: /CARD_BUS_0_SPI.~{CS}2 -> /CARD_BUS_1_SPI.~{CS}2
- U4 pad 1: /CARD_BUS_1_SPI.CARD_SEL -> /CARD_BUS_0_SPI.CARD_SEL
- U4 pad 10: /Card Bus Connectors1/CARD_CS.~{CS}2 -> /Card Bus Connectors0/F_CARD_CS.~{CS}2
- U4 pad 11: /Card Bus Connectors1/CARD_CS.~{CS}2 -> /Card Bus Connectors0/L_CARD_CS.~{CS}2
- U4 pad 2: /Card Bus Connectors1/CARD_CS.~{CS}0 -> /Card Bus Connectors0/L_CARD_CS.~{CS}0
- U4 pad 3: /Card Bus Connectors1/CARD_CS.~{CS}0 -> /Card Bus Connectors0/F_CARD_CS.~{CS}0
- U4 pad 4: /CARD_BUS_1_SPI.~{CS}0 -> /CARD_BUS_0_SPI.~{CS}0
- U4 pad 5: /Card Bus Connectors1/CARD_CS.~{CS}1 -> /Card Bus Connectors0/L_CARD_CS.~{CS}1
- U4 pad 6: /Card Bus Connectors1/CARD_CS.~{CS}1 -> /Card Bus Connectors0/F_CARD_CS.~{CS}1
- U4 pad 7: /CARD_BUS_1_SPI.~{CS}1 -> /CARD_BUS_0_SPI.~{CS}1
- U4 pad 9: /CARD_BUS_1_SPI.~{CS}2 -> /CARD_BUS_0_SPI.~{CS}2
- U5 pad 10: /Card Bus Connectors2/CARD_CS.~{CS}2 -> /Card Bus Connectors2/F_CARD_CS.~{CS}2
- U5 pad 11: /Card Bus Connectors2/CARD_CS.~{CS}2 -> /Card Bus Connectors2/L_CARD_CS.~{CS}2
- U5 pad 2: /Card Bus Connectors2/CARD_CS.~{CS}0 -> /Card Bus Connectors2/L_CARD_CS.~{CS}0
- U5 pad 3: /Card Bus Connectors2/CARD_CS.~{CS}0 -> /Card Bus Connectors2/F_CARD_CS.~{CS}0
- U5 pad 5: /Card Bus Connectors2/CARD_CS.~{CS}1 -> /Card Bus Connectors2/L_CARD_CS.~{CS}1
- U5 pad 6: /Card Bus Connectors2/CARD_CS.~{CS}1 -> /Card Bus Connectors2/F_CARD_CS.~{CS}1
- U6 pad 10: /Card Bus Connectors3/CARD_CS.~{CS}2 -> /Card Bus Connectors3/F_CARD_CS.~{CS}2
- U6 pad 11: /Card Bus Connectors3/CARD_CS.~{CS}2 -> /Card Bus Connectors3/L_CARD_CS.~{CS}2
- U6 pad 2: /Card Bus Connectors3/CARD_CS.~{CS}0 -> /Card Bus Connectors3/L_CARD_CS.~{CS}0
- U6 pad 3: /Card Bus Connectors3/CARD_CS.~{CS}0 -> /Card Bus Connectors3/F_CARD_CS.~{CS}0
- U6 pad 5: /Card Bus Connectors3/CARD_CS.~{CS}1 -> /Card Bus Connectors3/L_CARD_CS.~{CS}1
- U6 pad 6: /Card Bus Connectors3/CARD_CS.~{CS}1 -> /Card Bus Connectors3/F_CARD_CS.~{CS}1
- U7 pad 24: /EthernetInterface/~{RST} -> /~{MCU_RST}
Routing:
- net /CARD_BUS_0_SPI.~{DRDY}: track 0.00 -> 137.3 mm
- net /CARD_BUS_0_SPI.MISO: track 0.00 -> 135.5 mm, vias 0 -> 2
- net /CARD_BUS_0_SPI.MOSI: track 0.00 -> 134.9 mm, vias 0 -> 2
- net /CARD_BUS_0_SPI.SCLK: track 0.00 -> 134.5 mm, vias 0 -> 2
- net /CARD_BUS_0_SPI.~{CS}2: track 0.00 -> 111.8 mm, vias 0 -> 2
- net /CARD_BUS_0_SPI.CARD_SEL: track 0.00 -> 107.5 mm, vias 0 -> 2
- net /CARD_BUS_0_SPI.~{CS}1: track 0.00 -> 105.6 mm, vias 0 -> 2
- net /CARD_BUS_0_SPI.~{CS}0: track 0.00 -> 104.6 mm, vias 0 -> 2
- net /Card Bus Connectors0/~{RESET}: track 0.00 -> 75.0 mm
- net /8.192MHZ_CLK: track 0.00 -> 75.0 mm
- net +3.3V: track 10.7 -> 77.3 mm, vias 0 -> 16
- net GND: track 7.30 -> 71.3 mm, vias 28 -> 51
- net /CARD_BUS_1_SPI.CARD_SEL: track 0.00 -> 61.3 mm, vias 0 -> 2
- net /CARD_BUS_1_SPI.~{DRDY}: track 0.00 -> 58.8 mm, vias 0 -> 2
- net /CARD_BUS_1_SPI.MISO: track 0.00 -> 58.5 mm, vias 0 -> 2
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- added copper zone on In2.Cu, net +3.3V
- added copper zone on In1.Cu, net GND
Other:
- board outline added: 244.5 x 91 mm
- board text added: "MCU Rx"
- board text added: "MCU Tx"
- board text added: "Port 0.0"
- board text added: "Port 0.1"
- board text added: "Port 1.0"
- board text added: "Port 1.1"
- board text added: "UART Activity LEDs"

Commit message: Route most of the data lines on the PCB
Parts:
- removed the R15 at (193.3, 312.5)
- added D6: ESDS304, Package_TO_SOT_SMD:SOT-23-5, F.Cu at (149.2, 64.2)
- moved R2 321.5 mm to (123.2, 64.8), turned to 180 degrees
- moved C20 320.3 mm to (123.2, 63.0), turned to 180 degrees
- moved SW2 317.8 mm to (124.0, 60.0)
- moved R1 274.4 mm to (148.0, 108.0), turned to 180 degrees
- moved FB6 270.4 mm to (162.0, 52.2), turned to -90 degrees
- moved C19 267.7 mm to (148.0, 110.0), turned to 180 degrees
- moved D1 267.7 mm to (151.5, 107.5)
- moved TP1 264.2 mm to (156.2, 100.2)
- moved C14 264.1 mm to (142.0, 105.2), turned to -90 degrees
- moved R25 258.9 mm to (137.5, 47.2), turned to -90 degrees
- moved SW1 258.7 mm to (145.8, 115.8)
- moved FB1 256.0 mm to (160.2, 63.2), turned to 90 degrees
- moved R34 253.8 mm to (179.8, 66.8)
- moved R27 252.6 mm to (159.5, 47.2), turned to -90 degrees
- moved R26 248.8 mm to (139.5, 47.2), turned to -90 degrees
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Connections:
- R12 pad 6: Net-(J10-DAT1) -> Net-(J10-DAT2)
- R12 pad 7: Net-(J10-DAT2) -> Net-(J10-DAT1)
Routing:
- net /CARD_BUS_3_SPI.MOSI: track 0.00 -> 133.3 mm, vias 0 -> 1
- net /CARD_BUS_3_SPI.MISO: track 0.00 -> 132.3 mm
- net /CARD_BUS_3_SPI.CARD_SEL: track 0.00 -> 126.4 mm, vias 0 -> 2
- net /CARD_BUS_3_SPI.~{DRDY}: track 0.00 -> 117.6 mm, vias 0 -> 1
- net /CARD_BUS_3_SPI.SCLK: track 0.00 -> 109.8 mm, vias 0 -> 1
- net /CARD_BUS_3_SPI.~{CS}0: track 0.00 -> 104.2 mm, vias 0 -> 2
- net /CARD_BUS_3_SPI.~{CS}2: track 0.00 -> 103.7 mm, vias 0 -> 2
- net /CARD_BUS_3_SPI.~{CS}1: track 0.00 -> 101.6 mm
- net /Card Bus Connectors0/~{SYNC}: track 50.0 -> 150.1 mm
- net /~{ETH_SPEED_LED}: track 0.00 -> 78.8 mm, vias 0 -> 4
- net /8.192MHZ_CLK: track 75.0 -> 150.9 mm, vias 0 -> 1
- net /Card Bus Connectors0/~{RESET}: track 75.0 -> 150.0 mm
- net /CARD_BUS_2_SPI.CARD_SEL: track 0.00 -> 65.4 mm, vias 0 -> 4
- net /CARD_BUS_2_SPI.~{CS}0: track 0.00 -> 62.6 mm, vias 0 -> 2
- net /Card Bus Connectors3/L_CARD_CS.~{CS}0: track 0.00 -> 62.4 mm, vias 0 -> 2
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Other:
- board text added: "ISP Mode"
- board text added: "MCU UART USB"
- board text added: "Port 2.0"
- board text added: "Port 2.1"
- board text added: "Port 3.0"
- board text added: "Port 3.1"
- board text added: "Reset"
- board text added: "Rx"
- board text added: "SWD"
- board text added: "Tx"
- board text added: "V_{CORE}"
- board text removed: "MCU Rx"
- board text removed: "MCU Tx"
- board text removed: "UART Activity LEDs"

Commit message: Add schematic for Vsupply input
Parts:
- removed the R10 at (220.8, 53.4)
- removed the R11 at (220.8, 55.9)
- added C55: 100nF, Capacitor_SMD:C_0603_1608Metric, F.Cu at (8.79, 59.3)
- added C56: 10µF, Capacitor_SMD:C_1206_3216Metric, F.Cu at (22.2, 64.0)
- added D7: SMF24A, Diode_SMD:D_SMF, F.Cu at (16.6, 64.0)
- added J14: PJ-063AH, Connector_BarrelJack:BarrelJack_CUI_PJ-063AH_Horizontal, F.Cu at (19.0, 50.5)
- added J15: 0039300020, Project Library:Molex_Mini-Fit_Jr_5569-02A2_2x01_P4.20mm_Horizontal, F.Cu at (36.0, 52.5)
- added R43: .0025, Project Library:D1FCP0612, F.Cu at (8.68, 71.0)
- added R44: 10, Resistor_SMD:R_0603_1608Metric, F.Cu at (8.79, 61.8)
- added R45: 10, Resistor_SMD:R_0603_1608Metric, F.Cu at (8.79, 64.3)
- added TP2: +3.3VA, TestPoint:TestPoint_THTPad_D2.5mm_Drill1.2mm, F.Cu at (48.8, 25.9)
- added TP3: +3.3V, TestPoint:TestPoint_THTPad_D2.5mm_Drill1.2mm, F.Cu at (48.8, 30.4)
- added U15: INA180A3, Package_TO_SOT_SMD:SOT-23-5, F.Cu at (9.36, 68.0)
- R9: footprint Resistor_SMD:R_1206_3216Metric -> Resistor_SMD:R_0603_1608Metric
- moved LG1 145.0 mm to (116.4, 105.9)
- moved C52 64.9 mm to (162.0, 88.0), turned to -90 degrees
- moved D5 61.8 mm to (81.8, 43.8)
- moved R37 60.5 mm to (81.8, 39.8), turned to 180 degrees
- moved X2 59.1 mm to (159.0, 88.0)
- moved C30 23.6 mm to (193.8, 45.8)
- moved C32 20.6 mm to (195.5, 54.8), turned to 180 degrees
- moved C28 18.6 mm to (190.8, 54.8), turned to -90 degrees
- moved R10 18.3 mm to (189.2, 54.8), turned to 90 degrees
- moved C33 16.5 mm to (192.0, 58.5), turned to -90 degrees
- moved U8 14.7 mm to (195.0, 50.0), turned to 90 degrees
- moved R9 14.7 mm to (189.2, 43.2)
- moved U2 8.92 mm to (87.2, 31.0)
Connections:
- C51 pad 1: Net-(U12-+) -> Net-(U12--)
- C51 pad 2: Net-(U12--) -> Net-(U12-+)
- R39 pad 2: Net-(U12--) -> Net-(U12-+)
- R40 pad 2: Net-(U12-+) -> Net-(U12--)
- R9 pad 1: +3.3V -> /MicroSDCard/DET_A
- R9 pad 2: /MicroSDCard/DET_A -> +3.3V
- U1 pad 39: unconnected-(U1E-P4_17-Pad39) -> /V_{SUPPLY}_CUR_SENSE
Routing:
- net /Card Bus Connectors0/~{SYNC}: track 150.1 -> 246.9 mm, vias 0 -> 4
- net /8.192MHZ_CLK: track 150.9 -> 245.3 mm, vias 1 -> 4
- net /Card Bus Connectors0/~{RESET}: track 150.0 -> 242.7 mm, vias 0 -> 5
- net /MicroSDCard/+3.3V@SD: track 4.43 -> 45.3 mm, vias 0 -> 3
- net /CARD_BUS_2_SPI.~{DRDY}: track 30.5 -> 55.5 mm
- net +3.3V: track 108.2 -> 125.1 mm, vias 32 -> 34
- net /MicroSDCard/DET_B: track 0.00 -> 14.8 mm
- net GND: track 124.8 -> 133.2 mm, vias 75 -> 84
- net /MicroSDCard/DET_A: track 0.00 -> 2.84 mm
