File: hardware/Main Unit/Main Unit.kicad_pcb (KiCad board)
At the start: 4 copper layers, 244.5 x 91 mm, 153 parts, among them J1 3221-10-0300-00, J10 DM3AT, J11 USB4105-GF-A, J12 USB4105-GF-A, J13 HFJ11-2450E-L21RL, J14 PJ-063AH, J15 0039300020, J2 61801525123, J3 61801525123, J4 61801525123, J5 61801525123, J6 61801525123, J7 61801525123, J8 61801525123, J9 61801525123, SW1 MJTP1243, SW2 MJTP1243, U1 MCXN547VKLT, U10 USBLC6-2SC6, U11 TPS56A37RPAR, U12 INA180A3, U13 USBLC6-2SC6, U14 CY7C65223, U15 INA180A3, U2 TLV71333PDBV, U3 SN74CB3Q3257PWR, U4 SN74CB3Q3257PWR, U5 SN74CB3Q3257PWR, U6 SN74CB3Q3257PWR, U7 KSZ8081RND, U8 AP22913W6-7, U9 SN74AXC4T774, X1 24.0000MHz, X2 8.192MHz

Commit message: Route more of main unit, start on KiBot CI job
Parts:
- removed the R2 at (120.2, 6.51)
- removed the R3 at (70.0, 144.2)
- removed the R4 at (134.3, 283.6)
- added J16: 1x8, Connector_PinSocket_2.54mm:PinSocket_1x08_P2.54mm_Vertical, F.Cu at (175.8, 126.0)
- moved R18 277.5 mm to (130.2, 74.2), turned to 180 degrees
- moved R29 232.9 mm to (138.5, 70.8), turned to 180 degrees
- moved R28 225.9 mm to (138.5, 75.2), turned to 180 degrees
- moved TP2 118.3 mm to (124.8, 116.5)
- moved R3 110.3 mm to (141.5, 117.2), turned to 90 degrees
- moved C1 110.2 mm to (114.8, 116.5), turned to -90 degrees
- moved C2 108.3 mm to (121.5, 116.5), turned to -90 degrees
- moved R4 108.2 mm to (143.2, 117.2), turned to 90 degrees
- moved U2 90.9 mm to (118.0, 116.5), turned to 0 degrees
- moved C24 57.0 mm to (116.5, 95.5), turned to 180 degrees
- moved TP3 38.0 mm to (85.5, 40.2)
- moved R22 31.6 mm to (104.8, 55.5), turned to 90 degrees
- moved R24 26.2 mm to (104.8, 52.5), turned to 90 degrees
- moved U15 23.6 mm to (31.0, 58.5), turned to 180 degrees
- moved R45 22.5 mm to (28.0, 52.5)
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Connections:
- C55 pad 1: Net-(U15-V+) -> V_{SUPPLY}
- U1 pad 80: unconnected-(U1C-P0_4-Pad80) -> /MCU/MCU_P0_4
- U1 pad 81: unconnected-(U1C-P0_5-Pad81) -> /MCU/MCU_P0_5
- U1 pad 84: unconnected-(U1C-P0_16-Pad84) -> /MCU/MCU_P0_16
- U1 pad 85: unconnected-(U1C-P0_17-Pad85) -> /MCU/MCU_P0_17
- U1 pad 86: unconnected-(U1C-P0_18-Pad86) -> /MCU/MCU_P0_18
- U1 pad 87: unconnected-(U1C-P0_19-Pad87) -> /MCU/MCU_P0_19
- U1 pad 88: unconnected-(U1C-P0_20-Pad88) -> /MCU/MCU_P0_20
- U1 pad 89: unconnected-(U1C-P0_21-Pad89) -> /MCU/MCU_P0_21
- U15 pad 5: Net-(U15-V+) -> V_{SUPPLY}
Routing:
- net V_{SUPPLY}: track 18.0 -> 279.1 mm, vias 0 -> 11
- net /MCU/MCU_P0_4: track 0.00 -> 93.5 mm, vias 0 -> 2
- net /MCU/MCU_P0_5: track 0.00 -> 93.1 mm, vias 0 -> 2
- net /MCU/MCU_P0_16: track 0.00 -> 88.6 mm, vias 0 -> 2
- net /MCU/MCU_P0_17: track 0.00 -> 87.7 mm, vias 0 -> 2
- net /MCU/MCU_P0_18: track 0.00 -> 83.8 mm, vias 0 -> 2
- net /MCU/MCU_P0_19: track 0.00 -> 82.6 mm, vias 0 -> 2
- net /MCU/MCU_P0_20: track 0.00 -> 78.1 mm, vias 0 -> 2
- net /~{SD_CARD_EN}: track 0.00 -> 75.1 mm, vias 0 -> 4
- net /DBG_UART.MCU_TX: track 0.00 -> 72.1 mm, vias 0 -> 4
- net /MCU/MCU_P0_21: track 0.00 -> 71.3 mm, vias 0 -> 2
- net /MCU/USBMCU_VBUS: track 17.7 -> 83.1 mm, vias 0 -> 2
- net /DBG_UART.MCU_RX: track 0.00 -> 65.0 mm, vias 0 -> 4
- net /~{MCU_RST}: track 43.6 -> 103.4 mm, vias 0 -> 6
- net /MCU/USBMCU_D+: track 0.00 -> 58.9 mm, vias 0 -> 2
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Other:
- board text added: "+"
- board text added: "+3.3VA"
- board text added: "-"
- board text added: "Expansion Header (Direct Connection to MCU Pins)"
- board text added: "MCU Internal USB"
- board text added: "Mating Connector P/N: 0039013025"
- board text added: "P0_16"
- board text added: "P0_17"
- board text added: "P0_18"
- board text added: "P0_19"
- board text added: "P0_20"
- board text added: "P0_21"
- board text added: "P0_4"
- board text added: "P0_5"
- board text added: "V_{SUPPLY} Inputs +9-24Vdc Center Positive"
