File: hardware/Main Unit/EthernetInterface.kicad_sch (KiCad schematic)
At the start: 23 parts, among them J11 HFJ11-2450E-L21RL, U5 KSZ8081RND

Commit message: Update main unit to KiCAD 10, add clock buffer
Parts:
- J11: footprint Project Library:RJ45_HALO_HFJ11-x2450E-LxxRL_Horizontal-Fixed3DModel -> Connector_RJ:RJ45_HALO_HFJ11-x2450E-LxxRL_Horizontal
Connections:
- no-connect marks 2 -> 3

Commit message: Oops forgot to save
Parts:
- C28: renamed from C26; KiLib_Generator (none) -> Digi-Key
- C29: renamed from C27; KiLib_Generator (none) -> Digi-Key
- C31: renamed from C29; KiLib_Generator (none) -> Digi-Key
- C33: renamed from C31; KiLib_Generator (none) -> Digi-Key
- C34: renamed from C33; KiLib_Generator (none) -> Digi-Key
- C35: renamed from C32; KiLib_Generator (none) -> Digi-Key
- C44: renamed from C42; KiLib_Generator (none) -> Digi-Key
- C45: renamed from C43; KiLib_Generator (none) -> Digi-Key
- D6, FB1, FB2, R14, R17, R18, R19, R20, R22: KiLib_Generator (none) -> Digi-Key
- R16: renamed from R15; KiLib_Generator (none) -> Digi-Key
- R52: renamed from R54; KiLib_Generator (none) -> Digi-Key
- R53: renamed from R55; KiLib_Generator (none) -> Digi-Key
- R54: renamed from R56; KiLib_Generator (none) -> Digi-Key
- U7: renamed from U5; KiLib_Generator (none) -> Digi-Key
