File: hardware/Main Unit/EthernetInterface.kicad_sch (KiCad schematic)
At the start: 23 parts, among them J11 HFJ11-2450E-L21RL, U7 KSZ8081RND

Commit message: Update voltage card to KiCAD 10
Parts:
- J11: footprint Connector_RJ:RJ45_HALO_HFJ11-x2450E-LxxRL_Horizontal -> Project Library:RJ45_HALO_HFJ11-x2450E-LxxRL_Horizontal-Fixed3DModel
Changed lines of the file:
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@@
 			)
 		)
-		(property "Footprint" "Connector_RJ:RJ45_HALO_HFJ11-x2450E-LxxRL_Horizontal"
+		(property "Footprint" "Project Library:RJ45_HALO_HFJ11-x2450E-LxxRL_Horizontal-Fixed3DModel"
 			(at 210.82 56.515 0)
 			(hide yes)
