File: hardware/Main Unit/SupplyTo3.3VRegulator.kicad_sch (KiCad schematic)
At the start: 22 parts, among them U11 TPS56A37RPAR, U12 INA180A3

Commit message: Geographical reannotate
Parts:
- renumbered C48 to C49, C49 to C50, C50 to C52, C47 to C53, C51 to C57, C43 to C60, C44 to C61, C45 to C62, C46 to C65, D5 to D8, L2 to L3, R37 to R31, R31 to R37, R38 to R41, R35 to R42, R32 to R43, R36 to R48, R33 to R49, R40 to R52, R39 to R53, U12 to U15, U11 to U16
Changed lines of the file:
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@@
 		(dnp no)
 		(fields_autoplaced yes)
-		(property "Reference" "U11"
+		(property "Reference" "U16"
 			(at 125.73 52.07 0)
 			(effects
@@
 			(project "HackerDAQ Main Unit"
 				(path "/7d91f165-331a-4c48-9d02-ee2a0aa7e94a/6442a2f9-4c7d-4126-b24b-6ddb5831f5c5"
-					(reference "U11")
+					(reference "U16")
 					(unit 1)
 				)
@@
 		(on_board yes)
 		(dnp no)
-		(property "Reference" "R35"
+		(property "Reference" "R42"
 			(at 180.086 75.438 0)
 			(effects
@@
 			(project "HackerDAQ Main Unit"
 				(path "/7d91f165-331a-4c48-9d02-ee2a0aa7e94a/6442a2f9-4c7d-4126-b24b-6ddb5831f5c5"
-					(reference "R35")
+					(reference "R42")
 					(unit 1)
 				)
@@
 		(on_board yes)
 		(dnp no)
-		(property "Reference" "R40"
+		(property "Reference" "R52"
 			(at 221.742 88.646 0)
 			(effects
@@
 			(project "HackerDAQ Main Unit"
 				(path "/7d91f165-331a-4c48-9d02-ee2a0aa7e94a/6442a2f9-4c7d-4126-b24b-6ddb5831f5c5"
-					(reference "R40")
+					(reference "R52")
 					(unit 1)
 				)
@@
 		(dnp no)
 		(fields_autoplaced yes)
-		(property "Reference" "R38"
+		(property "Reference" "R41"
 			(at 218.44 62.23 90)
 			(effects
@@
 			(project "HackerDAQ Main Unit"
 				(path "/7d91f165-331a-4c48-9d02-ee2a0aa7e94a/6442a2f9-4c7d-4126-b24b-6ddb5831f5c5"
-					(reference "R38")
+					(reference "R41")
 					(unit 1)
 				)
@@
 		(on_board yes)
 		(dnp no)
-		(property "Reference" "R36"
+		(property "Reference" "R48"
 			(at 168.402 84.836 0)
 			(effects
@@
 			(project "HackerDAQ Main Unit"
 				(path "/7d91f165-331a-4c48-9d02-ee2a0aa7e94a/6442a2f9-4c7d-4126-b24b-6ddb5831f5c5"
-					(reference "R36")
+					(reference "R48")
 					(unit 1)
 				)
@@
 		(on_board yes)
 		(dnp no)
-		(property "Reference" "R39"
+		(property "Reference" "R53"
 			(at 211.582 88.646 0)
 			(effects
@@
 			(project "HackerDAQ Main Unit"
 				(path "/7d91f165-331a-4c48-9d02-ee2a0aa7e94a/6442a2f9-4c7d-4126-b24b-6ddb5831f5c5"
-					(reference "R39")
+					(reference "R53")
 					(unit 1)
 				)
@@
 		(on_board yes)
 		(dnp no)
-		(property "Reference" "C49"
+		(property "Reference" "C50"
 			(at 163.83 74.9235 0)
 			(effects
@@
 			(project "HackerDAQ Main Unit"
 				(path "/7d91f165-331a-4c48-9d02-ee2a0aa7e94a/6442a2f9-4c7d-4126-b24b-6ddb5831f5c5"
-					(reference "C49")
+					(reference "C50")
 					(unit 1)
 				)
@@
 		(dnp no)
 		(fields_autoplaced yes)
-		(property "Reference" "C45"
+		(property "Reference" "C62"
 			(at 73.66 63.5062 0)
 			(effects
@@
 			(project "HackerDAQ Main Unit"
 				(path "/7d91f165-331a-4c48-9d02-ee2a0aa7e94a/6442a2f9-4c7d-4126-b24b-6ddb5831f5c5"
-					(reference "C45")
+					(reference "C62")
 					(unit 1)
 				)
@@
 		(dnp no)
 		(fields_autoplaced yes)
-		(property "Reference" "C46"
+		(property "Reference" "C65"
 			(at 152.4063 54.61 90)
 			(effects
@@
 			(project "HackerDAQ Main Unit"
 				(path "/7d91f165-331a-4c48-9d02-ee2a0aa7e94a/6442a2f9-4c7d-4126-b24b-6ddb5831f5c5"
-					(reference "C46")
+					(reference "C65")
 					(unit 1)
 				)
@@
 		(on_board yes)
 		(dnp no)
-		(property "Reference" "R33"
+		(property "Reference" "R49"
 			(at 94.234 74.168 0)
 			(effects
@@
 			(project "HackerDAQ Main Unit"
 				(path "/7d91f165-331a-4c48-9d02-ee2a0aa7e94a/6442a2f9-4c7d-4126-b24b-6ddb5831f5c5"
-					(reference "R33")
+					(reference "R49")
 					(unit 1)
 				)
@@
 		(on_board yes)
 		(dnp no)
-		(property "Reference" "C47"
+		(property "Reference" "C53"
 			(at 187.96 72.3836 0)
 			(effects
@@
 			(project "HackerDAQ Main Unit"
 				(path "/7d91f165-331a-4c48-9d02-ee2a0aa7e94a/6442a2f9-4c7d-4126-b24b-6ddb5831f5c5"
-					(reference "C47")
+					(reference "C53")
 					(unit 1)
 				)
@@
 		(on_board yes)
 		(dnp no)
-		(property "Reference" "R31"
+		(property "Reference" "R37"
 			(at 99.314 95.758 0)
 			(effects
@@
 			(project "HackerDAQ Main Unit"
 				(path "/7d91f165-331a-4c48-9d02-ee2a0aa7e94a/6442a2f9-4c7d-4126-b24b-6ddb5831f5c5"
-					(reference "R31")
+					(reference "R37")
 					(unit 1)
 				)
@@
 		(dnp no)
 		(fields_autoplaced yes)
-		(property "Reference" "C48"
+		(property "Reference" "C49"
 			(at 198.12 72.3836 0)
 			(effects
@@
 			(project "HackerDAQ Main Unit"
 				(path "/7d91f165-331a-4c48-9d02-ee2a0aa7e94a/6442a2f9-4c7d-4126-b24b-6ddb5831f5c5"
-					(reference "C48")
+					(reference "C49")
 					(unit 1)
 				)
@@
 		(dnp no)
 		(fields_autoplaced yes)
-		(property "Reference" "D5"
+		(property "Reference" "D8"
 			(at 261.62 86.6774 90)
 			(effects
@@
 			(project "HackerDAQ Main Unit"
 				(path "/7d91f165-331a-4c48-9d02-ee2a0aa7e94a/6442a2f9-4c7d-4126-b24b-6ddb5831f5c5"
-					(reference "D5")
+					(reference "D8")
 					(unit 1)
 				)
@@
 		(dnp no)
 		(fields_autoplaced yes)
-		(property "Reference" "C50"
+		(property "Reference" "C52"
 			(at 240.03 101.6062 0)
 			(effects
@@
 			(project "HackerDAQ Main Unit"
 				(path "/7d91f165-331a-4c48-9d02-ee2a0aa7e94a/6442a2f9-4c7d-4126-b24b-6ddb5831f5c5"
-					(reference "C50")
+					(reference "C52")
 					(unit 1)
 				)
@@
 		(on_board yes)
 		(dnp no)
-		(property "Reference" "R37"
+		(property "Reference" "R31"
 			(at 255.27 78.994 90)
 			(effects
@@
 			(project "HackerDAQ Main Unit"
 				(path "/7d91f165-331a-4c48-9d02-ee2a0aa7e94a/6442a2f9-4c7d-4126-b24b-6ddb5831f5c5"
-					(reference "R37")
+					(reference "R31")
 					(unit 1)
 				)
@@
 		(on_board yes)
 		(dnp no)
-		(property "Reference" "R32"
+		(property "Reference" "R43"
 			(at 94.234 64.008 0)
 			(effects
@@
 			(project "HackerDAQ Main Unit"
 				(path "/7d91f165-331a-4c48-9d02-ee2a0aa7e94a/6442a2f9-4c7d-4126-b24b-6ddb5831f5c5"
-					(reference "R32")
+					(reference "R43")
 					(unit 1)
 				)
@@
 		(dnp no)
 		(fields_autoplaced yes)
-		(property "Reference" "C44"
+		(property "Reference" "C61"
 			(at 52.07 63.4936 0)
 			(effects
@@
 			(project "HackerDAQ Main Unit"
 				(path "/7d91f165-331a-4c48-9d02-ee2a0aa7e94a/6442a2f9-4c7d-4126-b24b-6ddb5831f5c5"
-					(reference "C44")
+					(reference "C61")
 					(unit 1)
 				)
@@
 		(dnp no)
 		(fields_autoplaced yes)
-		(property "Reference" "C43"
+		(property "Reference" "C60"
 			(at 62.23 63.4936 0)
 			(effects
@@
 			(project "HackerDAQ Main Unit"
 				(path "/7d91f165-331a-4c48-9d02-ee2a0aa7e94a/6442a2f9-4c7d-4126-b24b-6ddb5831f5c5"
-					(reference "C43")
+					(reference "C60")
 					(unit 1)
 				)
@@
 		(dnp no)
 		(fields_autoplaced yes)
-		(property "Reference" "L2"
+		(property "Reference" "L3"
 			(at 163.83 63.5 90)
 			(effects
@@
 			(project "HackerDAQ Main Unit"
 				(path "/7d91f165-331a-4c48-9d02-ee2a0aa7e94a/6442a2f9-4c7d-4126-b24b-6ddb5831f5c5"
-					(reference "L2")
+					(reference "L3")
 					(unit 1)
 				)
@@
 		(on_board yes)
 		(dnp no)
-		(property "Reference" "U12"
+		(property "Reference" "U15"
 			(at 234.696 111.506 0)
 			(effects
@@
 			(project "HackerDAQ Main Unit"
 				(path "/7d91f165-331a-4c48-9d02-ee2a0aa7e94a/6442a2f9-4c7d-4126-b24b-6ddb5831f5c5"
-					(reference "U12")
+					(reference "U15")
 					(unit 1)
 				)
@@
 		(dnp no)
 		(fields_autoplaced yes)
-		(property "Reference" "C51"
+		(property "Reference" "C57"
 			(at 218.4336 96.52 90)
 			(effects
@@
 			(project "HackerDAQ Main Unit"
 				(path "/7d91f165-331a-4c48-9d02-ee2a0aa7e94a/6442a2f9-4c7d-4126-b24b-6ddb5831f5c5"
-					(reference "C51")
-					(unit 1)
-				)
+					(reference "C57")
+					(unit 1)
+				)
