File: hardware/Main Unit/VsupplyInput.kicad_sch (KiCad schematic)
At the start: 9 parts, among them J14 PJ-063AH, J15 0039300020, U15 INA180A3

Commit message: Route more of main unit, start on KiBot CI job
Connections:
- net V_{SUPPLY}: now also C55.1, U15.5 (V+)
Changed lines of the file:
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@@
+	)
+	(junction
+		(at 157.48 99.06)
+		(diameter 0)
+		(color 0 0 0 0)
 	)
 	(junction
@@
 		(color 0 0 0 0)
 	)
+	(junction
+		(at 157.48 73.66)
+		(diameter 0)
+		(color 0 0 0 0)
+	)
 	(wire
 		(pts
@@
 	(wire
 		(pts
+			(xy 157.48 73.66) (xy 160.02 73.66)
+		)
+		(stroke
+			(width 0)
+			(type default)
+		)
+	)
+	(wire
+		(pts
 			(xy 147.32 101.6) (xy 147.32 91.44)
 		)
@@
 	(wire
 		(pts
-			(xy 147.32 73.66) (xy 160.02 73.66)
-		)
-		(stroke
+			(xy 147.32 73.66) (xy 157.48 73.66)
+		)
+		(stroke
+			(width 0)
+			(type default)
+		)
+	)
+	(wire
+		(pts
+			(xy 157.48 73.66) (xy 157.48 99.06)
+		)
+		(stroke

Commit message: Add LEDs and 5V regulator to main unit
Changed lines of the file:
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@@
-	)
-	(junction
-		(at 111.76 73.66)
-		(diameter 0)
-		(color 0 0 0 0)
 	)
 	(junction
@@
 	)
 	(junction
+		(at 111.76 96.52)
+		(diameter 0)
+		(color 0 0 0 0)
+	)
+	(junction
 		(at 147.32 101.6)
 		(diameter 0)
@@
 	)
 	(junction
+		(at 154.94 73.66)
+		(diameter 0)
+		(color 0 0 0 0)
+	)
+	(junction
 		(at 105.41 96.52)
 		(diameter 0)
@@
 	(wire
 		(pts
-			(xy 116.84 73.66) (xy 111.76 73.66)
-		)
-		(stroke
-			(width 0)
-			(type default)
-		)
-	)
-	(wire
-		(pts
 			(xy 157.48 110.49) (xy 157.48 99.06)
 		)
@@
 	(wire
 		(pts
+			(xy 111.76 96.52) (xy 105.41 96.52)
+		)
+		(stroke
+			(width 0)
+			(type default)
+		)
+	)
+	(wire
+		(pts
 			(xy 137.16 101.6) (xy 137.16 91.44)
 		)
@@
 	(wire
 		(pts
-			(xy 111.76 73.66) (xy 105.41 73.66)
+			(xy 105.41 73.66) (xy 116.84 73.66)
 		)
 		(stroke
@@
 	(wire
 		(pts
+			(xy 154.94 73.66) (xy 157.48 73.66)
+		)
+		(stroke
+			(width 0)
+			(type default)
+		)
+	)
+	(wire
+		(pts
 			(xy 116.84 73.66) (xy 137.16 73.66)
 		)
@@
 	(wire
 		(pts
-			(xy 147.32 73.66) (xy 157.48 73.66)
+			(xy 147.32 73.66) (xy 154.94 73.66)
 		)
 		(stroke
@@
 	(wire
 		(pts
-			(xy 116.84 96.52) (xy 105.41 96.52)
+			(xy 116.84 96.52) (xy 111.76 96.52)
 		)
 		(stroke
@@
 			)
 		)
-		(property "Description" "Resistor 10 ohm 1% 0.1W 0603"
+		(property "Description" "Resistor, small US symbol"
 			(at 147.32 88.9 0)
 			(effects
@@
 		)
 		(instances
-			(project "Main Unit"
+			(project "HackerDAQ Main Unit"
 				(path "/7d91f165-331a-4c48-9d02-ee2a0aa7e94a/9eb93347-9bc7-4661-8139-b1f7e57aefa1"
 					(reference "R45")
@@
 		)
 		(instances
-			(project "Main Unit"
+			(project "HackerDAQ Main Unit"
 				(path "/7d91f165-331a-4c48-9d02-ee2a0aa7e94a/9eb93347-9bc7-4661-8139-b1f7e57aefa1"
 					(reference "#PWR0148")
@@
 		)
 		(instances
-			(project "Main Unit"
+			(project "HackerDAQ Main Unit"
 				(path "/7d91f165-331a-4c48-9d02-ee2a0aa7e94a/9eb93347-9bc7-4661-8139-b1f7e57aefa1"
 					(reference "#PWR0147")
@@
 			)
 		)
-		(property "Datasheet" "https://www.littelfuse.com/assetdocs/tvs-diodes-smf-datasheet?assetguid=7eb8a5b6-bdd0-4561-8f19-0c3cc6f9b2af"
+		(property "Datasheet" "https://www.vishay.com/doc?85881"
 			(at 116.84 82.55 0)
 			(effects
@@
 			)
 		)
-		(property "Description" "200W unidirectional TVS diode, Vr=24V, Vbreakdown=29.5V"
+		(property "Description" "200W unidirectional Transil Transient Voltage Suppressor, 11Vrwm, SMF"
 			(at 116.84 83.82 0)
 			(effects
@@
 		)
 		(instances
-			(project "Main Unit"
+			(project "HackerDAQ Main Unit"
 				(path "/7d91f165-331a-4c48-9d02-ee2a0aa7e94a/9eb93347-9bc7-4661-8139-b1f7e57aefa1"
 					(reference "D7")
@@
 		)
 		(instances
-			(project "Main Unit"
+			(project "HackerDAQ Main Unit"
 				(path "/7d91f165-331a-4c48-9d02-ee2a0aa7e94a/9eb93347-9bc7-4661-8139-b1f7e57aefa1"
 					(reference "C55")
@@
 			)
 		)
-		(property "Datasheet" "https://mm.digikey.com/Volume0/opasdata/d220001/medias/docus/6239/D1FCP%20Series%20TFT-DMS-404-1.pdf"
+		(property "Datasheet" "~"
 			(at 142.24 73.66 0)
 			(effects
@@
 			)
 		)
-		(property "Description" "Current Sense Resistor 2.5mohm 1% 1W 0612"
+		(property "Description" "Shunt resistor with Kelvin connections, US symbol"
 			(at 142.24 73.66 0)
 			(effects
@@
 		)
 		(instances
-			(project "Main Unit"
+			(project "HackerDAQ Main Unit"
 				(path "/7d91f165-331a-4c48-9d02-ee2a0aa7e94a/9eb93347-9bc7-4661-8139-b1f7e57aefa1"
 					(reference "R43")
@@
 	(symbol
 		(lib_id "power:PWR_FLAG")
-		(at 111.76 73.66 0)
+		(at 154.94 73.66 0)
 		(unit 1)
 		(exclude_from_sim no)
@@
 		(fields_autoplaced yes)
 		(property "Reference" "#FLG04"
-			(at 111.76 71.755 0)
+			(at 154.94 71.755 0)
 			(effects
 				(font
@@
 		)
 		(property "Value" "PWR_FLAG"
-			(at 111.76 68.58 0)
+			(at 154.94 68.58 0)
 			(effects
 				(font
@@
 		)
 		(property "Footprint" ""
-			(at 111.76 73.66 0)
+			(at 154.94 73.66 0)
 			(effects
 				(font
@@
 		)
 		(property "Datasheet" "~"
-			(at 111.76 73.66 0)
+			(at 154.94 73.66 0)
 			(effects
 				(font
@@
 		)
 		(property "Description" "Special symbol for telling ERC where power comes from"
-			(at 111.76 73.66 0)
+			(at 154.94 73.66 0)
 			(effects
 				(font
@@
 		)
 		(instances
-			(project ""
+			(project "HackerDAQ Main Unit"
 				(path "/7d91f165-331a-4c48-9d02-ee2a0aa7e94a/9eb93347-9bc7-4661-8139-b1f7e57aefa1"
 					(reference "#FLG04")
@@
 		)
 		(instances
-			(project ""
+			(project "HackerDAQ Main Unit"
 				(path "/7d91f165-331a-4c48-9d02-ee2a0aa7e94a/9eb93347-9bc7-4661-8139-b1f7e57aefa1"
 					(reference "J15")
@@
 			)
 		)
-		(property "Description" "Resistor 10 ohm 1% 0.1W 0603"
+		(property "Description" "Resistor, small US symbol"
 			(at 137.16 88.9 0)
 			(effects
@@
 		)
 		(instances
-			(project "Main Unit"
+			(project "HackerDAQ Main Unit"
 				(path "/7d91f165-331a-4c48-9d02-ee2a0aa7e94a/9eb93347-9bc7-4661-8139-b1f7e57aefa1"
 					(reference "R44")
@@
 			)
 		)
-		(property "Datasheet" "https://www.cuidevices.com/product/resource/pj-063ah.pdf"
+		(property "Datasheet" "~"
 			(at 96.52 86.106 0)
 			(effects
@@
 			)
 		)
-		(property "Description" "DC Barrel Jack, 8A, 2.1mm ID, 5.5mm OD, 8.85mm Depth"
+		(property "Description" "DC Barrel Jack"
 			(at 95.25 85.09 0)
 			(effects
@@
 		)
 		(instances
-			(project "Main Unit"
+			(project "HackerDAQ Main Unit"
 				(path "/7d91f165-331a-4c48-9d02-ee2a0aa7e94a/9eb93347-9bc7-4661-8139-b1f7e57aefa1"
 					(reference "J14")
@@
 		)
 		(instances
-			(project "Main Unit"
+			(project "HackerDAQ Main Unit"
 				(path "/7d91f165-331a-4c48-9d02-ee2a0aa7e94a/9eb93347-9bc7-4661-8139-b1f7e57aefa1"
 					(reference "#PWR0146")
@@
 		)
 		(instances
-			(project "Main Unit"
+			(project "HackerDAQ Main Unit"
 				(path "/7d91f165-331a-4c48-9d02-ee2a0aa7e94a/9eb93347-9bc7-4661-8139-b1f7e57aefa1"
 					(reference "U15")
+					(unit 1)
+				)
+			)
+		)
+	)
+	(symbol
+		(lib_id "power:PWR_FLAG")
+		(at 111.76 96.52 180)
+		(unit 1)
+		(exclude_from_sim no)
+		(in_bom yes)
+		(on_board yes)
+		(dnp no)
+		(property "Reference" "#FLG05"
+			(at 111.76 98.425 0)
+			(effects
+				(font
+					(size 1.27 1.27)
+				)
+				(hide yes)
+			)
+		)
+		(property "Value" "PWR_FLAG"
+			(at 113.284 101.092 0)
+			(effects
+				(font
+					(size 1.27 1.27)
+				)
+			)
+		)
+		(property "Footprint" ""
+			(at 111.76 96.52 0)
+			(effects
+				(font
+					(size 1.27 1.27)
+				)
+				(hide yes)
+			)
+		)
+		(property "Datasheet" "~"
+			(at 111.76 96.52 0)
+			(effects
+				(font
+					(size 1.27 1.27)
+				)
+				(hide yes)
+			)
+		)
+		(property "Description" "Special symbol for telling ERC where power comes from"
+			(at 111.76 96.52 0)
+			(effects
+				(font
+					(size 1.27 1.27)
+				)
+				(hide yes)
+			)
+		)
+		(pin "1"
+		)
+		(instances
+			(project "HackerDAQ Main Unit"
+				(path "/7d91f165-331a-4c48-9d02-ee2a0aa7e94a/9eb93347-9bc7-4661-8139-b1f7e57aefa1"
+					(reference "#FLG05")
 					(unit 1)
 				)
@@
 		)
 		(instances
-			(project "Main Unit"
+			(project "HackerDAQ Main Unit"
 				(path "/7d91f165-331a-4c48-9d02-ee2a0aa7e94a/9eb93347-9bc7-4661-8139-b1f7e57aefa1"
 					(reference "C56")

Commit message: Main board routed!!
Parts:
- J14: symbol Connector:Barrel_Jack -> Connector:Barrel_Jack_MountingPin
Connections:
- no-connect marks 0 -> 1
Changed lines of the file:
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@@
 		(color 0 0 0 0)
+	)
+	(no_connect
+		(at 95.25 92.71)
 	)
 	(wire
@@
 	)
 	(symbol
-		(lib_id "Connector:Barrel_Jack")
+		(lib_id "Connector:Barrel_Jack_MountingPin")
 		(at 95.25 85.09 0)
 		(unit 1)
@@
 			)
 		)
-		(property "Description" "DC Barrel Jack"
+		(property "Description" "DC Barrel Jack with a mounting pin"
 			(at 95.25 85.09 0)
 			(effects
@@
 		(pin "1"
 		)
+		(pin "MP"
+		)
 		(instances

Commit message: Geographical reannotate
Parts:
- renumbered C55 to C40, C56 to C48, D7 to D9, J15 to J12, J14 to J13, R43 to R27, R45 to R36, R44 to R40, U15 to U10
Changed lines of the file:
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@@
 		(on_board yes)
 		(dnp no)
-		(property "Reference" "R45"
+		(property "Reference" "R36"
 			(at 145.542 87.376 0)
 			(effects
@@
 			(project "HackerDAQ Main Unit"
 				(path "/7d91f165-331a-4c48-9d02-ee2a0aa7e94a/9eb93347-9bc7-4661-8139-b1f7e57aefa1"
-					(reference "R45")
+					(reference "R36")
 					(unit 1)
 				)
@@
 		(dnp no)
 		(fields_autoplaced yes)
-		(property "Reference" "D7"
+		(property "Reference" "D9"
 			(at 119.38 82.5499 90)
 			(effects
@@
 			(project "HackerDAQ Main Unit"
 				(path "/7d91f165-331a-4c48-9d02-ee2a0aa7e94a/9eb93347-9bc7-4661-8139-b1f7e57aefa1"
-					(reference "D7")
+					(reference "D9")
 					(unit 1)
 				)
@@
 		(dnp no)
 		(fields_autoplaced yes)
-		(property "Reference" "C55"
+		(property "Reference" "C40"
 			(at 166.37 102.8762 0)
 			(effects
@@
 			(project "HackerDAQ Main Unit"
 				(path "/7d91f165-331a-4c48-9d02-ee2a0aa7e94a/9eb93347-9bc7-4661-8139-b1f7e57aefa1"
-					(reference "C55")
+					(reference "C40")
 					(unit 1)
 				)
@@
 		(on_board yes)
 		(dnp no)
-		(property "Reference" "R43"
+		(property "Reference" "R27"
 			(at 138.938 70.104 90)
 			(effects
@@
 			(project "HackerDAQ Main Unit"
 				(path "/7d91f165-331a-4c48-9d02-ee2a0aa7e94a/9eb93347-9bc7-4661-8139-b1f7e57aefa1"
-					(reference "R43")
+					(reference "R27")
 					(unit 1)
 				)
@@
 		(dnp no)
 		(fields_autoplaced yes)
-		(property "Reference" "J15"
+		(property "Reference" "J12"
 			(at 72.39 83.5659 90)
 			(effects
@@
 			(project "HackerDAQ Main Unit"
 				(path "/7d91f165-331a-4c48-9d02-ee2a0aa7e94a/9eb93347-9bc7-4661-8139-b1f7e57aefa1"
-					(reference "J15")
+					(reference "J12")
 					(unit 1)
 				)
@@
 		(on_board yes)
 		(dnp no)
-		(property "Reference" "R44"
+		(property "Reference" "R40"
 			(at 135.382 87.376 0)
 			(effects
@@
 			(project "HackerDAQ Main Unit"
 				(path "/7d91f165-331a-4c48-9d02-ee2a0aa7e94a/9eb93347-9bc7-4661-8139-b1f7e57aefa1"
-					(reference "R44")
+					(reference "R40")
 					(unit 1)
 				)
@@
 		(dnp no)
 		(fields_autoplaced yes)
-		(property "Reference" "J14"
+		(property "Reference" "J13"
 			(at 95.25 76.2 0)
 			(effects
@@
 			(project "HackerDAQ Main Unit"
 				(path "/7d91f165-331a-4c48-9d02-ee2a0aa7e94a/9eb93347-9bc7-4661-8139-b1f7e57aefa1"
-					(reference "J14")
+					(reference "J13")
 					(unit 1)
 				)
@@
 		(on_board yes)
 		(dnp no)
-		(property "Reference" "U15"
+		(property "Reference" "U10"
 			(at 161.036 112.776 0)
 			(effects
@@
 			(project "HackerDAQ Main Unit"
 				(path "/7d91f165-331a-4c48-9d02-ee2a0aa7e94a/9eb93347-9bc7-4661-8139-b1f7e57aefa1"
-					(reference "U15")
+					(reference "U10")
 					(unit 1)
 				)
@@
 		(dnp no)
 		(fields_autoplaced yes)
-		(property "Reference" "C56"
+		(property "Reference" "C48"
 			(at 142.2336 95.25 90)
 			(effects
@@
 			(project "HackerDAQ Main Unit"
 				(path "/7d91f165-331a-4c48-9d02-ee2a0aa7e94a/9eb93347-9bc7-4661-8139-b1f7e57aefa1"
-					(reference "C56")
-					(unit 1)
-				)
+					(reference "C48")
+					(unit 1)
+				)
