File: hardware/Main Unit/VsupplyInput.kicad_sch (KiCad schematic)
At the start: 9 parts, among them J12 0039300020, J13 PJ-063AH, U10 INA180A3

Commit message: Oops forgot to save
Parts:
- C42: renamed from C40; KiLib_Generator (none) -> Digi-Key
- C50: renamed from C48; KiLib_Generator (none) -> Digi-Key
- R36, R40: KiLib_Generator (none) -> Digi-Key
- U12: renamed from U10; KiLib_Generator (none) -> Digi-Key
Changed lines of the file:
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@@
+			)
+		)
+		(property "KiLib_Generator" "Digi-Key"
+			(at 147.32 88.9 0)
+			(hide yes)
+			(show_name no)
+			(do_not_autoplace no)
+			(effects
+				(font
+					(size 1.27 1.27)
+				)
 			)
 		)
@@
 		(dnp no)
 		(fields_autoplaced yes)
-		(property "Reference" "C40"
+		(property "Reference" "C42"
 			(at 166.37 102.8762 0)
 			(show_name no)
@@
 		)
 		(property "LibRef" "ESD35C104K4T2A-24"
+			(at 163.83 104.14 0)
+			(hide yes)
+			(show_name no)
+			(do_not_autoplace no)
+			(effects
+				(font
+					(size 1.27 1.27)
+				)
+			)
+		)
+		(property "KiLib_Generator" "Digi-Key"
 			(at 163.83 104.14 0)
 			(hide yes)
@@
 			(project "HackerDAQ Main Unit"
 				(path "/7d91f165-331a-4c48-9d02-ee2a0aa7e94a/9eb93347-9bc7-4661-8139-b1f7e57aefa1"
-					(reference "C40")
+					(reference "C42")
 					(unit 1)
 				)
@@
 			)
 		)
+		(property "KiLib_Generator" "Digi-Key"
+			(at 137.16 88.9 0)
+			(hide yes)
+			(show_name no)
+			(do_not_autoplace no)
+			(effects
+				(font
+					(size 1.27 1.27)
+				)
+			)
+		)
 		(pin "2"
 		)
@@
 		(in_pos_files yes)
 		(dnp no)
-		(property "Reference" "U10"
+		(property "Reference" "U12"
 			(at 161.036 112.776 0)
 			(show_name no)
@@
 		)
 		(property "SKU" "296-47654-1-ND"
+			(at 160.02 118.11 0)
+			(hide yes)
+			(show_name no)
+			(do_not_autoplace no)
+			(effects
+				(font
+					(size 1.27 1.27)
+				)
+			)
+		)
+		(property "KiLib_Generator" "Digi-Key"
 			(at 160.02 118.11 0)
 			(hide yes)
@@
 			(project "HackerDAQ Main Unit"
 				(path "/7d91f165-331a-4c48-9d02-ee2a0aa7e94a/9eb93347-9bc7-4661-8139-b1f7e57aefa1"
-					(reference "U10")
+					(reference "U12")
 					(unit 1)
 				)
@@
 		(dnp no)
 		(fields_autoplaced yes)
-		(property "Reference" "C48"
+		(property "Reference" "C50"
 			(at 142.2336 95.25 90)
 			(show_name no)
@@
 		)
 		(property "LibRef" "CL31B106KLHNNNE"
+			(at 142.24 101.6 0)
+			(hide yes)
+			(show_name no)
+			(do_not_autoplace no)
+			(effects
+				(font
+					(size 1.27 1.27)
+				)
+			)
+		)
+		(property "KiLib_Generator" "Digi-Key"
 			(at 142.24 101.6 0)
 			(hide yes)
@@
 			(project "HackerDAQ Main Unit"
 				(path "/7d91f165-331a-4c48-9d02-ee2a0aa7e94a/9eb93347-9bc7-4661-8139-b1f7e57aefa1"
-					(reference "C48")
+					(reference "C50")
 					(unit 1)
 				)
