File: hardware/Main Unit/HackerDAQ Main Unit.kicad_pcb (KiCad board)
At the start: 4 copper layers, 244.5 x 91 mm, 151 parts, among them J1 3221-10-0300-00, J10 DM3AT, J11 USB4105-GF-A, J12 USB4105-GF-A, J13 HFJ11-2450E-L21RL, J14 PJ-063AH, J15 0039300020, J16 1x8, J2 61801525123, J3 61801525123, J4 61801525123, J5 61801525123, J6 61801525123, J7 61801525123, J8 61801525123, J9 61801525123, SW1 MJTP1243, SW2 MJTP1243, U1 MCXN547VKLT, U10 USBLC6-2SC6, U11 TPS56A37RPAR, U12 INA180A3, U13 USBLC6-2SC6, U14 CY7C65223, U15 INA180A3, U2 TLV71333PDBV, U3 SN74CB3Q3257PWR, U4 SN74CB3Q3257PWR, U5 SN74CB3Q3257PWR, U6 SN74CB3Q3257PWR, U7 KSZ8081RND, U8 AP22913W6-7, U9 SN74AXC4T774, X1 24.0000MHz, X2 8.192MHz

Commit message: Add LEDs and 5V regulator to main unit
Parts:
- added C57: 10µF, Capacitor_SMD:C_1210_3225Metric, F.Cu at (50.2, 12.4)
- added C58: 10µF, Capacitor_SMD:C_1210_3225Metric, F.Cu at (50.2, 16.7)
- added C59: 100nF, Capacitor_SMD:C_0603_1608Metric, F.Cu at (55.1, 11.6)
- added C60: 100nF, Capacitor_SMD:C_0603_1608Metric, F.Cu at (55.1, 14.1)
- added C61: 150pF, Capacitor_SMD:C_0603_1608Metric, F.Cu at (55.1, 16.6)
- added C62: 22µF, Capacitor_SMD:C_1210_3225Metric, F.Cu at (50.2, 20.9)
- added C63: 22µF, Capacitor_SMD:C_1210_3225Metric, F.Cu at (50.2, 25.2)
- added C64: 10µF, Capacitor_SMD:C_1206_3216Metric, F.Cu at (50.2, 29.0)
- added C65: 100nF, Capacitor_SMD:C_0603_1608Metric, F.Cu at (55.1, 19.1)
- added D10: AA3528SURSK, ColorLEDs:AA3528, F.Cu at (42.4, 12.5)
- added D11: AA3528QBS, ColorLEDs:AA3528, F.Cu at (42.4, 17.2)
- added D8: AA3528CGSK, ColorLEDs:AA3528, F.Cu at (67.2, 28.2)
- added D9: ASMB-MTB0-0A3A2, LED_SMD:LED_Avago_PLCC4_3.2x2.8mm_CW, F.Cu at (50.5, 34.9)
- added L3: 3.3μH, Inductor_SMD:L_Vishay_IHLP-3232, F.Cu at (58.7, 25.2)
- added R46: 18.2k, Resistor_SMD:R_0603_1608Metric, F.Cu at (59.1, 11.6)
- added R47: 3.01k, Resistor_SMD:R_0603_1608Metric, F.Cu at (59.1, 14.1)
- added R48: 52.3k, Resistor_SMD:R_0603_1608Metric, F.Cu at (59.1, 16.6)
- added R49: 10k, Resistor_SMD:R_0603_1608Metric, F.Cu at (59.1, 19.1)
- added R50: 73.2k, Resistor_SMD:R_0603_1608Metric, F.Cu at (63.1, 11.6)
- added R51: 10, Resistor_SMD:R_0603_1608Metric, F.Cu at (63.1, 14.1)
- added R52: .0025, Project Library:D1FCP0612, F.Cu at (67.0, 15.8)
- added R53: 10, Resistor_SMD:R_0603_1608Metric, F.Cu at (63.1, 16.6)
- added R54: 270, Resistor_SMD:R_0603_1608Metric, F.Cu at (63.1, 19.1)
- added R55: 30, Resistor_SMD:R_0603_1608Metric, F.Cu at (37.5, 11.5)
- added R56: 30, Resistor_SMD:R_0603_1608Metric, F.Cu at (37.5, 14.0)
- added R57: 140, Resistor_SMD:R_0603_1608Metric, F.Cu at (37.5, 16.5)
- added R58: 30, Resistor_SMD:R_0603_1608Metric, F.Cu at (37.5, 19.0)
- added R59: 140, Resistor_SMD:R_0603_1608Metric, F.Cu at (37.5, 21.5)
- added TP4: +5V, TestPoint:TestPoint_THTPad_D2.5mm_Drill1.2mm, F.Cu at (57.8, 35.0)
- added U16: TPS56A37RPAR, Project Library:RPA0010A-MFG, F.Cu at (67.4, 23.1)
- added U17: INA180A3, Package_TO_SOT_SMD:SOT-23-5, F.Cu at (67.7, 12.7)
- J13: footprint Project Library:RJ45_HALO_HFJ11-x2450E-LxxRL_Horizontal-Fixed3DModel -> Connector_RJ:RJ45_HALO_HFJ11-x2450E-LxxRL_Horizontal
- U7: footprint Project Library:QFN-24-1EP_4x4mm_P0.5mm_EP2.65x2.65mm-LengthenedPads -> Package_DFN_QFN:QFN-24-1EP_4x4mm_P0.5mm_EP2.6x2.6mm
Connections:
- U1 pad 22: unconnected-(U1E-P4_0-Pad22) -> /+3.3V_CUR_SENSE
- U1 pad 23: unconnected-(U1E-P4_1-Pad23) -> /MCU/+5V_CUR_SENSE
- U1 pad 24: unconnected-(U1E-P4_2-Pad24) -> /V_{SUPPLY}_CUR_SENSE
- U1 pad 25: unconnected-(U1E-P4_3-Pad25) -> /MCU/STATUS_LED
- U1 pad 26: unconnected-(U1E-P4_4-Pad26) -> /MCU/ERROR_LED
- U1 pad 37: /+3.3V_CUR_SENSE -> /MCU/RGB_LED_~{R}
- U1 pad 38: /MCU/+5V_CUR_SENSE -> /MCU/RGB_LED_~{G}
- U1 pad 39: /V_{SUPPLY}_CUR_SENSE -> /MCU/RGB_LED_~{B}
Routing:
- net /V_{SUPPLY}_CUR_SENSE: track 48.5 -> 0.00 mm, vias 1 -> 0
- net /MCU/RGB_LED_~{B}: track 0.00 -> 48.5 mm, vias 0 -> 1
- net /MCU/RGB_LED_~{G}: track 0.00 -> 46.8 mm, vias 0 -> 1
- net /MCU/+5V_CUR_SENSE: track 46.8 -> 0.00 mm, vias 1 -> 0
- net /MCU/RGB_LED_~{R}: track 0.00 -> 45.0 mm, vias 0 -> 1
- net /+3.3V_CUR_SENSE: track 45.0 -> 0.00 mm, vias 1 -> 0

Commit message: Main board routed!!
Parts:
- added H1: MountingHole_Pad, MountingHole:MountingHole_4.3mm_M4_DIN965_Pad, F.Cu at (251.8, 98.0)
- added H2: MountingHole_Pad, MountingHole:MountingHole_4.3mm_M4_DIN965_Pad, F.Cu at (251.8, 17.0)
- added H3: MountingHole_Pad, MountingHole:MountingHole_4.3mm_M4_DIN965_Pad, F.Cu at (17.2, 98.0)
- added H4: MountingHole_Pad, MountingHole:MountingHole_4.3mm_M4_DIN965_Pad, F.Cu at (17.2, 17.0)
- D9: value ASMB-MTB0-0A3A2 -> ASMB-MTB0-0B3A2; footprint LED_SMD:LED_Avago_PLCC4_3.2x2.8mm_CW -> ColorLEDs:LED_Avago_PLCC4_3.2x2.8mm_CW_Fixed3DModel
- J13: footprint Connector_RJ:RJ45_HALO_HFJ11-x2450E-LxxRL_Horizontal -> Project Library:RJ45_HALO_HFJ11-x2450E-LxxRL_Horizontal-Fixed3DModel
- X1, X2: footprint Oscillator:Oscillator_SMD_ECS_2520MV-xxx-xx-4Pin_2.5x2.0mm -> Project Library:Oscillator_SMD_ECS_2520MV-xxx-xx-4Pin_2.5x2.0mm_Fixed3DModel
- moved C23 227.0 mm to (235.8, 19.0), turned to 0 degrees
- moved J14 224.0 mm to (239.5, 89.8), turned to 0 degrees
- moved J4 222.9 mm to (245.2, 58.0), turned to -90 degrees
- moved D7 220.8 mm to (238.5, 86.0), turned to 180 degrees
- moved J9 219.7 mm to (25.2, 58.0), turned to -90 degrees
- moved R43 218.5 mm to (237.8, 83.0), turned to 90 degrees
- moved U4 215.6 mm to (231.8, 23.8), turned to 0 degrees
- moved R6 209.0 mm to (231.8, 32.0), turned to -90 degrees
- moved R8 206.6 mm to (36.5, 37.0), turned to -90 degrees
- moved R44 206.1 mm to (230.5, 89.2), turned to 180 degrees
- moved R45 205.5 mm to (230.5, 87.8), turned to 180 degrees
- moved C55 205.3 mm to (231.2, 81.5), turned to -90 degrees
- moved C26 199.9 mm to (34.5, 66.8), turned to 0 degrees
- moved C56 198.9 mm to (227.5, 85.5), turned to 180 degrees
- moved U15 197.9 mm to (227.5, 81.8), turned to 0 degrees
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Connections:
- J14 pad MP: (no net) -> unconnected-(J14-MountPin-PadMP)_1
- R55 pad 2: /MCU/RGB_LED_~{R} -> /MCU/RGB_LED_~{B}
- R57 pad 2: /MCU/RGB_LED_~{B} -> /MCU/RGB_LED_~{R}
Routing:
- net +5V: track 0.00 -> 506.5 mm, vias 0 -> 5
- net /~{MCU_RST}: track 103.4 -> 315.9 mm, vias 6 -> 10
- net V_{SUPPLY}: track 279.1 -> 472.2 mm, vias 11 -> 19
- net /+3.3V_CUR_SENSE: track 0.00 -> 150.9 mm, vias 0 -> 2
- net /V_{SUPPLY}_CUR_SENSE: track 0.00 -> 113.1 mm, vias 0 -> 2
- net /MCU/+5V_CUR_SENSE: track 0.00 -> 86.9 mm, vias 0 -> 2
- net /MCU/MCU_P0_21: track 71.3 -> 139.5 mm, vias 2 -> 1
- net /MCU/STATUS_LED: track 0.00 -> 66.0 mm, vias 0 -> 2
- net /MCU/MCU_P0_20: track 78.1 -> 137.7 mm, vias 2 -> 1
- net /MCU/ERROR_LED: track 0.00 -> 59.4 mm, vias 0 -> 2
- net /MCU/MCU_P0_19: track 82.6 -> 135.4 mm, vias 2 -> 1
- net /MCU/MCU_P0_18: track 83.8 -> 133.5 mm, vias 2 -> 1
- net /MCU/MCU_P0_17: track 87.7 -> 133.2 mm, vias 2 -> 1
- net /MCU/MCU_P0_16: track 88.6 -> 132.9 mm, vias 2 -> 1
- net /MCU/MCU_P0_5: track 93.1 -> 132.2 mm, vias 2 -> 1
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- added copper zone on F.Cu, net +3.3V
- added copper zone on F.Cu, net +5V
- added copper zone on F.Cu, net /SupplyTo5VRegulator/SW
Other:
- board text added: "+3.3V"
- board text added: "+5V"
- board text added: "Activity"
- board text added: "Error"
- board text added: "Main Unit MCX N Rev 1rc1"
- board text added: "Status"

Commit message: Geographical reannotate
Parts:
- renumbered C25 to C1, C11 to C10, C18 to C11, C15 to C12, C16 to C13, C24 to C14, C12 to C15, C27 to C16, C6 to C17, C21 to C18, C13 to C19, C23 to C2, C8 to C20, C52 to C21, C9 to C22, C7 to C23, C5 to C24, C4 to C25, C42 to C26, C41 to C27, C26 to C28, C36 to C29, C2 to C3, C34 to C30, C35 to C31, C39 to C32, C40 to C33, C20 to C34, C53 to C35, C22 to C36, C54 to C37, C33 to C38, C29 to C39, C1 to C4, C55 to C40, C31 to C41, C37 to C42, C38 to C43, C32 to C44, C28 to C45, C63 to C46, C61 to C47, C56 to C48, C48 to C49, C19 to C5, C49 to C50, C62 to C51, C50 to C52, C47 to C53, C64 to C54, C58 to C55, C57 to C56, C51 to C57, C30 to C58, C14 to C6, C43 to C60, C44 to C61, C45 to C62, C65 to C63, C60 to C64, C46 to C65, C3 to C7, C17 to C8, C10 to C9, D11 to D1, D4 to D10, D3 to D11, D10 to D2, D9 to D3, D1 to D4, D2 to D5, D8 to D7, D5 to D8, D7 to D9, FB6 to FB2, H4 to H1, H1 to H4, J16 to J10, J13 to J11, J15 to J12, J14 to J13, J10 to J14, J12 to J15, J11 to J16, J9 to J2, J8 to J3, J7 to J4, J6 to J5, J3 to J6, J2 to J7, J5 to J8, J4 to J9, L3 to L2, L2 to L3, R58 to R1, R6 to R10, R8 to R11, R5 to R12, R7 to R13, R28 to R14, R17 to R15, R18 to R16, R16 to R17, R29 to R18, R13 to R19, R59 to R2, R14 to R20, R34 to R21, R30 to R22, R2 to R23, R12 to R24, R11 to R25, R54 to R26, R43 to R27, R10 to R28, R22 to R29, R57 to R3, R48 to R30, R37 to R31, R50 to R32, R46 to R33, R24 to R34, R52 to R35, R45 to R36, R31 to R37, R49 to R38, R47 to R39, R56 to R4, R44 to R40, R38 to R41, R35 to R42, R32 to R43, R41 to R44, R42 to R45, R53 to R46, R51 to R47, R36 to R48, R33 to R49, R4 to R5, R15 to R50, R19 to R51, R40 to R52, R39 to R53, R27 to R54, R26 to R55, R25 to R56, R20 to R57, R21 to R58, R9 to R59, R3 to R6, R55 to R7, R23 to R8, R1 to R9, TP2 to TP1, TP1 to TP2, TP4 to TP3, TP3 to TP4, U5 to U1, U15 to U10, U13 to U11, U10 to U12, U8 to U13, U16 to U14, U12 to U15, U11 to U16, U4 to U3, U1 to U4, U7 to U5, U3 to U6, U6 to U7, U14 to U8
