File: hardware/Main Unit/HackerDAQ Main Unit.kicad_pcb (KiCad board)
At the start: 4 copper layers, 244.5 x 91 mm, 186 parts, among them J1 3221-10-0300-00, J10 1x8, J11 HFJ11-2450E-L21RL, J12 0039300020, J13 PJ-063AH, J14 DM3AT, J15 USB4105-GF-A, J16 USB4105-GF-A, J2 61801525123, J3 61801525123, J4 61801525123, J5 61801525123, J6 61801525123, J7 61801525123, J8 61801525123, J9 61801525123, SW1 MJTP1243, SW2 MJTP1243, U1 SN74CB3Q3257PWR, U10 INA180A3, U11 USBLC6-2SC6, U12 USBLC6-2SC6, U13 AP22913W6-7, U14 TPS56A37RPAR, U15 INA180A3, U16 TPS56A37RPAR, U17 INA180A3, U2 TLV71333PDBV, U3 SN74CB3Q3257PWR, U4 MCXN547VKLT, U5 KSZ8081RND, U6 SN74CB3Q3257PWR, U7 SN74CB3Q3257PWR, U8 CY7C65223, U9 SN74AXC4T774, X1 24.0000MHz, X2 8.192MHz

Commit message: Update main unit to KiCAD 10, add clock buffer
Parts:
- added C12: 100nF, Capacitor_SMD:C_0603_1608Metric, F.Cu at (160.5, 39.0)
- added C25: 100nF, Capacitor_SMD:C_0603_1608Metric, F.Cu at (107.3, 58.5)
- added U4: SN74LVC1G34DBVR, Package_TO_SOT_SMD:SOT-23-5, F.Cu at (158.0, 43.2)
- added U6: SN74LVC1G34DBVR, Package_TO_SOT_SMD:SOT-23-5, F.Cu at (108.2, 54.8)
- D3: footprint ColorLEDs:LED_Avago_PLCC4_3.2x2.8mm_CW_Fixed3DModel -> LED_SMD:LED_Avago_PLCC4_3.2x2.8mm_CW
- J11: footprint Project Library:RJ45_HALO_HFJ11-x2450E-LxxRL_Horizontal-Fixed3DModel -> Connector_RJ:RJ45_HALO_HFJ11-x2450E-LxxRL_Horizontal
- X1, X2: footprint Project Library:Oscillator_SMD_ECS_2520MV-xxx-xx-4Pin_2.5x2.0mm_Fixed3DModel -> Oscillator:Oscillator_SMD_ECS_2520MV-xxx-xx-4Pin_2.5x2.0mm
- moved C22 7.87 mm to (114.6, 51.5), turned to -90 degrees
- moved X2 1.92 mm to (111.6, 51.5), turned to 0 degrees
- renumbered C12 to C13, C13 to C14, C14 to C15, C15 to C16, C16 to C17, C17 to C18, C18 to C19, C19 to C20, C20 to C21, C21 to C22, C22 to C23, C23 to C24, C24 to C26, C25 to C27, C26 to C28, C27 to C29, C28 to C30, C29 to C31, C30 to C32, C31 to C33, C33 to C34, C32 to C35, C34 to C36, C35 to C37, C36 to C38, C37 to C39, C39 to C40, C38 to C41, C40 to C42, C41 to C43, C42 to C44, C43 to C45, C44 to C46, C45 to C47, C46 to C48, C47 to C49, C48 to C50, C50 to C51, C49 to C52, C51 to C53, C52 to C54, C53 to C55, C55 to C56, C56 to C57, C54 to C58, C57 to C60, C58 to C61, C60 to C62, C61 to C63, C62 to C64, C63 to C65, C64 to C66, C65 to C67, R12 to R11, R11 to R12, R16 to R15, R15 to R16, R29 to R28, R28 to R29, R35 to R34, R34 to R35, R38 to R37, R39 to R38, R37 to R39, R42 to R41, R43 to R42, R44 to R43, R45 to R44, R41 to R45, R50 to R48, R51 to R49, R48 to R50, R49 to R51, R54 to R52, R55 to R53, R56 to R54, R52 to R55, R53 to R56, U8 to U10, U9 to U11, U10 to U12, U11 to U13, U12 to U14, U13 to U15, U14 to U16, U15 to U17, U16 to U18, U17 to U19, U4 to U5, U5 to U7, U6 to U8, U7 to U9
Connections:
- J2 pad 4: /8.192MHZ_CLK -> /8.192MHZ_CLK_L
- J3 pad 4: /8.192MHZ_CLK -> /8.192MHZ_CLK_L
- J4 pad 4: /8.192MHZ_CLK -> /8.192MHZ_CLK_L
- J5 pad 4: /8.192MHZ_CLK -> /8.192MHZ_CLK_L
- J6 pad 4: /8.192MHZ_CLK -> /8.192MHZ_CLK_R
- J7 pad 4: /8.192MHZ_CLK -> /8.192MHZ_CLK_R
- J8 pad 4: /8.192MHZ_CLK -> /8.192MHZ_CLK_R
- J9 pad 4: /8.192MHZ_CLK -> /8.192MHZ_CLK_R
Routing:
- net /8.192MHZ_CLK: track 246.2 -> 82.0 mm
- net /8.192MHZ_CLK_R: track 0.00 -> 88.6 mm, vias 0 -> 1
- net /8.192MHZ_CLK_L: track 0.00 -> 84.6 mm, vias 0 -> 1
- net GND: track 180.9 -> 187.5 mm, vias 127 -> 129
- net +3.3V: track 131.0 -> 136.2 mm, vias 43 -> 45

Commit message: Update voltage card to KiCAD 10
Parts:
- J11: footprint Connector_RJ:RJ45_HALO_HFJ11-x2450E-LxxRL_Horizontal -> Project Library:RJ45_HALO_HFJ11-x2450E-LxxRL_Horizontal-Fixed3DModel
Connections:
- J16 pad SH: unconnected-(J16-SHIELD-PadSH)_3 -> /DebugUSBUART/unconnected-(J16-SHIELD-PadSH)_3_3
