File: hardware/Main Unit/CardBusConnectors.kicad_sch (KiCad schematic)
At the start: 5 parts, among them J6 61801525123, J7 61801525123, U6 SN74CB3Q3257PWR

Commit message: Update main unit to KiCAD 10, add clock buffer
Connections:
- net GND: now also J6.SH (PAD), J7.SH (PAD); no longer J6.0 (PAD), J7.0 (PAD)

Commit message: Oops forgot to save
Parts:
- C38: renamed from C36; KiLib_Generator (none) -> Digi-Key
- U8: renamed from U6; KiLib_Generator (none) -> Digi-Key
- renumbered R12 to R11
Changed lines of the file:
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@@
 		(dnp no)
 		(fields_autoplaced yes)
-		(property "Reference" "R12"
+		(property "Reference" "R11"
 			(at 163.83 44.7039 0)
 			(show_name no)
@@
 			(project "HackerDAQ Main Unit"
 				(path "/7d91f165-331a-4c48-9d02-ee2a0aa7e94a/647fa122-ba55-4257-82a5-33756e3f8461"
+					(reference "R11")
+					(unit 1)
+				)
+				(path "/7d91f165-331a-4c48-9d02-ee2a0aa7e94a/65abad2d-a04a-4486-8762-5ae3bd8749b5"
 					(reference "R12")
-					(unit 1)
-				)
-				(path "/7d91f165-331a-4c48-9d02-ee2a0aa7e94a/65abad2d-a04a-4486-8762-5ae3bd8749b5"
-					(reference "R11")
 					(unit 1)
 				)
@@
 		(in_pos_files yes)
 		(dnp no)
-		(property "Reference" "U6"
+		(property "Reference" "U8"
 			(at 99.822 47.244 0)
 			(show_name no)
@@
 		(property "SKU" "296-19138-1-ND"
 			(at 152.908 25.146 0)
+			(hide yes)
+			(show_name no)
+			(do_not_autoplace no)
+			(effects
+				(font
+					(size 1.27 1.27)
+				)
+			)
+		)
+		(property "KiLib_Generator" "Digi-Key"
+			(at 114.3 67.31 0)
 			(hide yes)
 			(show_name no)
@@
 			(project "HackerDAQ Main Unit"
 				(path "/7d91f165-331a-4c48-9d02-ee2a0aa7e94a/647fa122-ba55-4257-82a5-33756e3f8461"
-					(reference "U6")
+					(reference "U8")
 					(unit 1)
 				)
 				(path "/7d91f165-331a-4c48-9d02-ee2a0aa7e94a/65abad2d-a04a-4486-8762-5ae3bd8749b5"
-					(reference "U7")
+					(reference "U9")
 					(unit 1)
 				)
@@
 		(in_pos_files yes)
 		(dnp no)
-		(property "Reference" "C36"
+		(property "Reference" "C38"
 			(at 115.57 38.1062 0)
 			(show_name no)
@@
 		)
 		(property "LibRef" "ESD35C104K4T2A-24"
+			(at 118.11 39.37 0)
+			(hide yes)
+			(show_name no)
+			(do_not_autoplace no)
+			(effects
+				(font
+					(size 1.27 1.27)
+				)
+			)
+		)
+		(property "KiLib_Generator" "Digi-Key"
 			(at 118.11 39.37 0)
 			(hide yes)
@@
 			(project "HackerDAQ Main Unit"
 				(path "/7d91f165-331a-4c48-9d02-ee2a0aa7e94a/647fa122-ba55-4257-82a5-33756e3f8461"
-					(reference "C36")
+					(reference "C38")
 					(unit 1)
 				)
 				(path "/7d91f165-331a-4c48-9d02-ee2a0aa7e94a/65abad2d-a04a-4486-8762-5ae3bd8749b5"
-					(reference "C28")
-					(unit 1)
-				)
+					(reference "C30")
+					(unit 1)
+				)
