File: hardware/Main Unit/DebugUSBUART.kicad_sch (KiCad schematic)
At the start: 14 parts, among them J16 USB4105-GF-A, U12 USBLC6-2SC6, U8 CY7C65223

Commit message: Oops forgot to save
Parts:
- C32: renamed from C30; KiLib_Generator (none) -> Digi-Key
- C37: renamed from C35; KiLib_Generator (none) -> Digi-Key
- C39: renamed from C37; KiLib_Generator (none) -> Digi-Key
- R28: renamed from R29; KiLib_Generator (none) -> Digi-Key
- R35: renamed from R34; KiLib_Generator (none) -> Digi-Key
- R48: renamed from R50; KiLib_Generator (none) -> Digi-Key
- R49: renamed from R51; KiLib_Generator (none) -> Digi-Key
- R57, R58: KiLib_Generator (none) -> Digi-Key
- U14: renamed from U12; KiLib_Generator (none) -> Digi-Key
- renumbered U8 to U10
Connections:
- net unconnected-(J16-SHIELD-PadSH)_3: now reaches J16.SH (SHIELD)
Changed lines of the file:
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@@
+		)
+	)
+	(label "unconnected-(J16-SHIELD-PadSH)_3"
+		(at 20.32 102.87 270)
+		(effects
+			(font
+				(size 1.27 1.27)
+			)
+			(justify right bottom)
 		)
 	)
@@
 		(dnp no)
 		(fields_autoplaced yes)
-		(property "Reference" "U8"
+		(property "Reference" "U10"
 			(at 130.81 52.07 0)
 			(show_name no)
@@
 			(project "HackerDAQ Main Unit"
 				(path "/7d91f165-331a-4c48-9d02-ee2a0aa7e94a/435dc57d-0a8b-4ccd-93d5-e5334c096ca6"
-					(reference "U8")
+					(reference "U10")
 					(unit 1)
 				)
@@
 		(in_pos_files yes)
 		(dnp no)
-		(property "Reference" "U12"
+		(property "Reference" "U14"
 			(at 66.294 72.136 0)
 			(show_name no)
@@
 		)
 		(property "LibRef" ""
+			(at 71.12 80.01 0)
+			(hide yes)
+			(show_name no)
+			(do_not_autoplace no)
+			(effects
+				(font
+					(size 1.27 1.27)
+				)
+			)
+		)
+		(property "KiLib_Generator" "Digi-Key"
 			(at 71.12 80.01 0)
 			(hide yes)
@@
 			(project "HackerDAQ Main Unit"
 				(path "/7d91f165-331a-4c48-9d02-ee2a0aa7e94a/435dc57d-0a8b-4ccd-93d5-e5334c096ca6"
-					(reference "U12")
+					(reference "U14")
 					(unit 1)
 				)
@@
 		(in_pos_files yes)
 		(dnp no)
-		(property "Reference" "R29"
+		(property "Reference" "R28"
 			(at 83.312 68.58 0)
 			(show_name no)
@@
 		)
 		(property "LibRef" "RC0603FR-0710KL"
+			(at 88.9 69.85 0)
+			(hide yes)
+			(show_name no)
+			(do_not_autoplace no)
+			(effects
+				(font
+					(size 1.27 1.27)
+				)
+			)
+		)
+		(property "KiLib_Generator" "Digi-Key"
 			(at 88.9 69.85 0)
 			(hide yes)
@@
 			(project "HackerDAQ Main Unit"
 				(path "/7d91f165-331a-4c48-9d02-ee2a0aa7e94a/435dc57d-0a8b-4ccd-93d5-e5334c096ca6"
-					(reference "R29")
+					(reference "R28")
 					(unit 1)
 				)
@@
 			)
 		)
+		(property "KiLib_Generator" "Digi-Key"
+			(at 198.12 81.28 0)
+			(hide yes)
+			(show_name no)
+			(do_not_autoplace no)
+			(effects
+				(font
+					(size 1.27 1.27)
+				)
+			)
+		)
 		(pin "2"
 		)
@@
 		(in_pos_files yes)
 		(dnp no)
-		(property "Reference" "R34"
+		(property "Reference" "R35"
 			(at 82.804 61.468 0)
 			(show_name no)
@@
 		)
 		(property "LibRef" "RC0603FR-074K7L"
+			(at 88.9 62.23 0)
+			(hide yes)
+			(show_name no)
+			(do_not_autoplace no)
+			(effects
+				(font
+					(size 1.27 1.27)
+				)
+			)
+		)
+		(property "KiLib_Generator" "Digi-Key"
 			(at 88.9 62.23 0)
 			(hide yes)
@@
 			(project "HackerDAQ Main Unit"
 				(path "/7d91f165-331a-4c48-9d02-ee2a0aa7e94a/435dc57d-0a8b-4ccd-93d5-e5334c096ca6"
-					(reference "R34")
+					(reference "R35")
 					(unit 1)
 				)
@@
 		(dnp no)
 		(fields_autoplaced yes)
-		(property "Reference" "C30"
+		(property "Reference" "C32"
 			(at 93.98 44.4562 0)
 			(show_name no)
@@
 		)
 		(property "LibRef" "ESD35C104K4T2A-24"
+			(at 91.44 45.72 0)
+			(hide yes)
+			(show_name no)
+			(do_not_autoplace no)
+			(effects
+				(font
+					(size 1.27 1.27)
+				)
+			)
+		)
+		(property "KiLib_Generator" "Digi-Key"
 			(at 91.44 45.72 0)
 			(hide yes)
@@
 			(project "HackerDAQ Main Unit"
 				(path "/7d91f165-331a-4c48-9d02-ee2a0aa7e94a/435dc57d-0a8b-4ccd-93d5-e5334c096ca6"
-					(reference "C30")
+					(reference "C32")
 					(unit 1)
 				)
@@
 			)
 		)
+		(property "KiLib_Generator" "Digi-Key"
+			(at 191.77 85.09 0)
+			(hide yes)
+			(show_name no)
+			(do_not_autoplace no)
+			(effects
+				(font
+					(size 1.27 1.27)
+				)
+			)
+		)
 		(pin "2"
 		)
@@
 		(in_pos_files yes)
 		(dnp no)
-		(property "Reference" "C37"
+		(property "Reference" "C39"
 			(at 93.726 55.88 0)
 			(show_name no)
@@
 		)
 		(property "LibRef" "CL10B105MO8NNWC"
+			(at 99.06 57.15 0)
+			(hide yes)
+			(show_name no)
+			(do_not_autoplace no)
+			(effects
+				(font
+					(size 1.27 1.27)
+				)
+			)
+		)
+		(property "KiLib_Generator" "Digi-Key"
 			(at 99.06 57.15 0)
 			(hide yes)
@@
 			(project "HackerDAQ Main Unit"
 				(path "/7d91f165-331a-4c48-9d02-ee2a0aa7e94a/435dc57d-0a8b-4ccd-93d5-e5334c096ca6"
-					(reference "C37")
+					(reference "C39")
 					(unit 1)
 				)
@@
 		(in_pos_files yes)
 		(dnp no)
-		(property "Reference" "R50"
+		(property "Reference" "R48"
 			(at 43.942 68.326 90)
 			(show_name no)
@@
 		(property "LibRef" "RC0603FR-075K1L"
 			(at 49.53 69.85 90)
+			(hide yes)
+			(show_name no)
+			(do_not_autoplace no)
+			(effects
+				(font
+					(size 1.27 1.27)
+				)
+			)
+		)
+		(property "KiLib_Generator" "Digi-Key"
+			(at 49.53 69.85 0)
 			(hide yes)
 			(show_name no)
@@
 			(project "HackerDAQ Main Unit"
 				(path "/7d91f165-331a-4c48-9d02-ee2a0aa7e94a/435dc57d-0a8b-4ccd-93d5-e5334c096ca6"
-					(reference "R50")
+					(reference "R48")
 					(unit 1)
 				)
@@
 		(dnp no)
 		(fields_autoplaced yes)
-		(property "Reference" "C35"
+		(property "Reference" "C37"
 			(at 104.14 44.4562 0)
 			(show_name no)
@@
 		)
 		(property "LibRef" "ESD35C104K4T2A-24"
+			(at 101.6 45.72 0)
+			(hide yes)
+			(show_name no)
+			(do_not_autoplace no)
+			(effects
+				(font
+					(size 1.27 1.27)
+				)
+			)
+		)
+		(property "KiLib_Generator" "Digi-Key"
 			(at 101.6 45.72 0)
 			(hide yes)
@@
 			(project "HackerDAQ Main Unit"
 				(path "/7d91f165-331a-4c48-9d02-ee2a0aa7e94a/435dc57d-0a8b-4ccd-93d5-e5334c096ca6"
-					(reference "C35")
+					(reference "C37")
 					(unit 1)
 				)
@@
 		(in_pos_files yes)
 		(dnp no)
-		(property "Reference" "R51"
+		(property "Reference" "R49"
 			(at 43.942 73.914 90)
 			(show_name no)
@@
 		(property "LibRef" "RC0603FR-075K1L"
 			(at 49.53 72.39 90)
+			(hide yes)
+			(show_name no)
+			(do_not_autoplace no)
+			(effects
+				(font
+					(size 1.27 1.27)
+				)
+			)
+		)
+		(property "KiLib_Generator" "Digi-Key"
+			(at 49.53 72.39 0)
 			(hide yes)
 			(show_name no)
@@
 			(project "HackerDAQ Main Unit"
 				(path "/7d91f165-331a-4c48-9d02-ee2a0aa7e94a/435dc57d-0a8b-4ccd-93d5-e5334c096ca6"
-					(reference "R51")
+					(reference "R49")
 					(unit 1)
 				)
