File: hardware/Main Unit/MCU.kicad_sch (KiCad schematic)
At the start: 49 parts, among them J1 3221-10-0300-00, J10 1x8, J15 USB4105-GF-A, SW1 MJTP1243, SW2 MJTP1243, U11 USBLC6-2SC6, U4 MCXN547VKLT, X1 24.0000MHz

Commit message: Update main unit to KiCAD 10, add clock buffer
Parts:
- D3: footprint ColorLEDs:LED_Avago_PLCC4_3.2x2.8mm_CW_Fixed3DModel -> LED_SMD:LED_Avago_PLCC4_3.2x2.8mm_CW
- X1: footprint Project Library:Oscillator_SMD_ECS_2520MV-xxx-xx-4Pin_2.5x2.0mm_Fixed3DModel -> Oscillator:Oscillator_SMD_ECS_2520MV-xxx-xx-4Pin_2.5x2.0mm

Commit message: Oops forgot to save
Parts:
- C10, C11, C5, C6, C7, C8, C9, D4, D5, J10, L1, R1, R2, R23, R3, R4, R5, R6, R7, R8, R9: KiLib_Generator (none) -> Digi-Key
- C13: renamed from C12; KiLib_Generator (none) -> Digi-Key
- C14: renamed from C13; KiLib_Generator (none) -> Digi-Key
- C15: renamed from C14; KiLib_Generator (none) -> Digi-Key
- C16: renamed from C15; KiLib_Generator (none) -> Digi-Key
- C17: renamed from C16; KiLib_Generator (none) -> Digi-Key
- C18: renamed from C17; KiLib_Generator (none) -> Digi-Key
- C19: renamed from C18; KiLib_Generator (none) -> Digi-Key
- C20: renamed from C19; KiLib_Generator (none) -> Digi-Key
- C21: renamed from C20; KiLib_Generator (none) -> Digi-Key
- C23: renamed from C22; KiLib_Generator (none) -> Digi-Key
- C24: renamed from C23; KiLib_Generator (none) -> Digi-Key
- C26: renamed from C24; KiLib_Generator (none) -> Digi-Key
- C27: renamed from C25; KiLib_Generator (none) -> Digi-Key
- C36: renamed from C34; KiLib_Generator (none) -> Digi-Key
- R15: renamed from R16; KiLib_Generator (none) -> Digi-Key
- R43: renamed from R44; KiLib_Generator (none) -> Digi-Key
- R44: renamed from R45; KiLib_Generator (none) -> Digi-Key
- U13: renamed from U11; KiLib_Generator (none) -> Digi-Key
- renumbered U4 to U5
