File: hardware/Main Unit/MicroSDCard.kicad_sch (KiCad schematic)
At the start: 14 parts, among them J14 DM3AT, U13 AP22913W6-7, U9 SN74AXC4T774

Commit message: Update main unit to KiCAD 10, add clock buffer
Connections:
- net GND: now also J14.SH (SHIELD); no longer J14.11 (SHIELD)

Commit message: Oops forgot to save
Parts:
- C40: renamed from C39; KiLib_Generator (none) -> Digi-Key
- C41: renamed from C38; KiLib_Generator (none) -> Digi-Key
- C43: renamed from C41; KiLib_Generator (none) -> Digi-Key
- C46: renamed from C44; KiLib_Generator (none) -> Digi-Key
- C47: renamed from C45; KiLib_Generator (none) -> Digi-Key
- C61: renamed from C58; KiLib_Generator (none) -> Digi-Key
- R21, R25, R59: KiLib_Generator (none) -> Digi-Key
- R29: renamed from R28; KiLib_Generator (none) -> Digi-Key
- U11: renamed from U9; KiLib_Generator (none) -> Digi-Key
- U15: renamed from U13; KiLib_Generator (none) -> Digi-Key
Changed lines of the file:
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@@
+			)
+		)
+		(property "KiLib_Generator" "Digi-Key"
+			(at 71.12 46.99 0)
+			(hide yes)
+			(show_name no)
+			(do_not_autoplace no)
+			(effects
+				(font
+					(size 1.27 1.27)
+				)
 			)
 		)
@@
 		(dnp no)
 		(fields_autoplaced yes)
-		(property "Reference" "U13"
+		(property "Reference" "U15"
 			(at 139.065 31.75 0)
 			(show_name no)
@@
 		(property "Supplier" "Digi-Key"
 			(at 136.398 68.834 0)
+			(hide yes)
+			(show_name no)
+			(do_not_autoplace no)
+			(effects
+				(font
+					(size 1.27 1.27)
+				)
+			)
+		)
+		(property "KiLib_Generator" "Digi-Key"
+			(at 135.89 46.99 0)
 			(hide yes)
 			(show_name no)
@@
 			(project "HackerDAQ Main Unit"
 				(path "/7d91f165-331a-4c48-9d02-ee2a0aa7e94a/171a326f-5e68-4f6e-be23-ff3df57281ba"
-					(reference "U13")
+					(reference "U15")
 					(unit 1)
 				)
@@
 			)
 		)
+		(property "KiLib_Generator" "Digi-Key"
+			(at 166.37 107.95 0)
+			(hide yes)
+			(show_name no)
+			(do_not_autoplace no)
+			(effects
+				(font
+					(size 1.27 1.27)
+				)
+			)
+		)
 		(pin "2"
 		)
@@
 		(in_pos_files yes)
 		(dnp no)
-		(property "Reference" "R28"
+		(property "Reference" "R29"
 			(at 108.204 51.054 0)
 			(show_name no)
@@
 		)
 		(property "LibRef" "RC0603FR-0710KL"
+			(at 106.68 52.07 0)
+			(hide yes)
+			(show_name no)
+			(do_not_autoplace no)
+			(effects
+				(font
+					(size 1.27 1.27)
+				)
+			)
+		)
+		(property "KiLib_Generator" "Digi-Key"
 			(at 106.68 52.07 0)
 			(hide yes)
@@
 			(project "HackerDAQ Main Unit"
 				(path "/7d91f165-331a-4c48-9d02-ee2a0aa7e94a/171a326f-5e68-4f6e-be23-ff3df57281ba"
-					(reference "R28")
+					(reference "R29")
 					(unit 1)
 				)
@@
 		(dnp no)
 		(fields_autoplaced yes)
-		(property "Reference" "U9"
+		(property "Reference" "U11"
 			(at 140.97 69.85 0)
 			(show_name no)
@@
 		)
 		(property "SKU" "296-SN74AXC4T774PWRCT-ND"
+			(at 140.97 93.98 0)
+			(hide yes)
+			(show_name no)
+			(do_not_autoplace no)
+			(effects
+				(font
+					(size 1.27 1.27)
+				)
+			)
+		)
+		(property "KiLib_Generator" "Digi-Key"
 			(at 140.97 93.98 0)
 			(hide yes)
@@
 			(project "HackerDAQ Main Unit"
 				(path "/7d91f165-331a-4c48-9d02-ee2a0aa7e94a/171a326f-5e68-4f6e-be23-ff3df57281ba"
-					(reference "U9")
+					(reference "U11")
 					(unit 1)
 				)
@@
 		(in_pos_files yes)
 		(dnp no)
-		(property "Reference" "C41"
+		(property "Reference" "C43"
 			(at 153.67 67.3162 0)
 			(show_name no)
@@
 		)
 		(property "LibRef" "CL10B105MO8NNWC"
+			(at 151.13 67.31 0)
+			(hide yes)
+			(show_name no)
+			(do_not_autoplace no)
+			(effects
+				(font
+					(size 1.27 1.27)
+				)
+			)
+		)
+		(property "KiLib_Generator" "Digi-Key"
 			(at 151.13 67.31 0)
 			(hide yes)
@@
 			(project "HackerDAQ Main Unit"
 				(path "/7d91f165-331a-4c48-9d02-ee2a0aa7e94a/171a326f-5e68-4f6e-be23-ff3df57281ba"
-					(reference "C41")
+					(reference "C43")
 					(unit 1)
 				)
@@
 		(in_pos_files yes)
 		(dnp no)
-		(property "Reference" "C39"
+		(property "Reference" "C40"
 			(at 115.57 73.6662 0)
 			(show_name no)
@@
 		)
 		(property "LibRef" "CL10B105MO8NNWC"
+			(at 113.03 73.66 0)
+			(hide yes)
+			(show_name no)
+			(do_not_autoplace no)
+			(effects
+				(font
+					(size 1.27 1.27)
+				)
+			)
+		)
+		(property "KiLib_Generator" "Digi-Key"
 			(at 113.03 73.66 0)
 			(hide yes)
@@
 			(project "HackerDAQ Main Unit"
 				(path "/7d91f165-331a-4c48-9d02-ee2a0aa7e94a/171a326f-5e68-4f6e-be23-ff3df57281ba"
-					(reference "C39")
+					(reference "C40")
 					(unit 1)
 				)
@@
 		(in_pos_files yes)
 		(dnp no)
-		(property "Reference" "C44"
+		(property "Reference" "C46"
 			(at 160.02 45.974 0)
 			(show_name no)
@@
 		)
 		(property "LibRef" "CL31B106KLHNNNE"
+			(at 153.67 46.99 0)
+			(hide yes)
+			(show_name no)
+			(do_not_autoplace no)
+			(effects
+				(font
+					(size 1.27 1.27)
+				)
+			)
+		)
+		(property "KiLib_Generator" "Digi-Key"
 			(at 153.67 46.99 0)
 			(hide yes)
@@
 			(project "HackerDAQ Main Unit"
 				(path "/7d91f165-331a-4c48-9d02-ee2a0aa7e94a/171a326f-5e68-4f6e-be23-ff3df57281ba"
-					(reference "C44")
+					(reference "C46")
 					(unit 1)
 				)
@@
 			)
 		)
+		(property "KiLib_Generator" "Digi-Key"
+			(at 114.3 109.22 0)
+			(hide yes)
+			(show_name no)
+			(do_not_autoplace no)
+			(effects
+				(font
+					(size 1.27 1.27)
+				)
+			)
+		)
 		(pin "2"
 		)
@@
 		(in_pos_files yes)
 		(dnp no)
-		(property "Reference" "C58"
+		(property "Reference" "C61"
 			(at 114.3 40.894 0)
 			(show_name no)
@@
 		)
 		(property "LibRef" "CL31B106KLHNNNE"
+			(at 120.65 41.91 0)
+			(hide yes)
+			(show_name no)
+			(do_not_autoplace no)
+			(effects
+				(font
+					(size 1.27 1.27)
+				)
+			)
+		)
+		(property "KiLib_Generator" "Digi-Key"
 			(at 120.65 41.91 0)
 			(hide yes)
@@
 			(project "HackerDAQ Main Unit"
 				(path "/7d91f165-331a-4c48-9d02-ee2a0aa7e94a/171a326f-5e68-4f6e-be23-ff3df57281ba"
-					(reference "C58")
+					(reference "C61")
 					(unit 1)
 				)
@@
 		(dnp no)
 		(fields_autoplaced yes)
-		(property "Reference" "C38"
+		(property "Reference" "C41"
 			(at 208.28 68.5862 0)
 			(show_name no)
@@
 		)
 		(property "LibRef" "ESD35C104K4T2A-24"
+			(at 205.74 69.85 0)
+			(hide yes)
+			(show_name no)
+			(do_not_autoplace no)
+			(effects
+				(font
+					(size 1.27 1.27)
+				)
+			)
+		)
+		(property "KiLib_Generator" "Digi-Key"
 			(at 205.74 69.85 0)
 			(hide yes)
@@
 			(project "HackerDAQ Main Unit"
 				(path "/7d91f165-331a-4c48-9d02-ee2a0aa7e94a/171a326f-5e68-4f6e-be23-ff3df57281ba"
-					(reference "C38")
+					(reference "C41")
 					(unit 1)
 				)
@@
 		(in_pos_files yes)
 		(dnp no)
-		(property "Reference" "C45"
+		(property "Reference" "C47"
 			(at 100.33 52.0762 0)
 			(show_name no)
@@
 		)
 		(property "LibRef" "CL10B105MO8NNWC"
+			(at 97.79 52.07 0)
+			(hide yes)
+			(show_name no)
+			(do_not_autoplace no)
+			(effects
+				(font
+					(size 1.27 1.27)
+				)
+			)
+		)
+		(property "KiLib_Generator" "Digi-Key"
 			(at 97.79 52.07 0)
 			(hide yes)
@@
 			(project "HackerDAQ Main Unit"
 				(path "/7d91f165-331a-4c48-9d02-ee2a0aa7e94a/171a326f-5e68-4f6e-be23-ff3df57281ba"
-					(reference "C45")
+					(reference "C47")
 					(unit 1)
 				)
