File: hardware/Common Sheets/B2B Connector Card Side.kicad_sch (KiCad schematic)
At the start: 1 part, among them J9 LD15S33E4GX00LF

Commit message: Finish redesigned DIO card
Parts:
- renumbered J9 to J6
Changed lines of the file:
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@@
 		(dnp no)
 		(fields_autoplaced yes)
-		(property "Reference" "J9"
+		(property "Reference" "J6"
 			(at 132.08 58.4199 0)
 			(effects
@@
 			(project ""
 				(path "/af2d881c-6553-449d-9093-6deb41497bdc/fd74a83f-66e8-460e-b889-0885a11eca86"
-					(reference "J9")
+					(reference "J6")
 					(unit 1)
 				)

Commit message: Route more of main unit, start on KiBot CI job
Parts:
- renumbered J6 to J9
Changed lines of the file:
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@@
 		(dnp no)
 		(fields_autoplaced yes)
-		(property "Reference" "J6"
+		(property "Reference" "J9"
 			(at 132.08 58.4199 0)
 			(effects
@@
 			)
 		)
-		(property "Datasheet" "https://cdn.amphenol-cs.com/media/wysiwyg/files/drawing/10130914.pdf"
+		(property "Datasheet" "~"
 			(at 127 59.69 0)
 			(effects
@@
 			(project ""
 				(path "/af2d881c-6553-449d-9093-6deb41497bdc/fd74a83f-66e8-460e-b889-0885a11eca86"
-					(reference "J6")
+					(reference "J9")
 					(unit 1)
 				)
