File: hardware/Common Sheets/B2B Connector Card Side.kicad_sch (KiCad schematic)
At the start: 1 part, among them J9 LD15S33E4GX00LF

Commit message: Fix DRC/ERC errors
Parts:
- renumbered J9 to J6
Changed lines of the file:
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@@
 		(dnp no)
 		(fields_autoplaced yes)
-		(property "Reference" "J9"
+		(property "Reference" "J6"
 			(at 132.08 58.4199 0)
 			(effects
@@
 			(project ""
 				(path "/af2d881c-6553-449d-9093-6deb41497bdc/fd74a83f-66e8-460e-b889-0885a11eca86"
-					(reference "J9")
+					(reference "J6")
 					(unit 1)
 				)

Commit message: Update voltage card to KiCAD 10
Connections:
- net GND: now also J6.SH (PAD); no longer J6.0 (PAD)
