File: hardware/Common Sheets/AD7770_ADC.kicad_sch (KiCad schematic)
At the start: 31 parts, among them U1 AD7770

Commit message: Route more of main unit, start on KiBot CI job
Parts:
- renumbered C23 to C10, C24 to C11, C21 to C12, C20 to C13, C27 to C15, C22 to C16, C25 to C17, C13 to C18, C17 to C20, C19 to C21, C18 to C22, C16 to C23, C10 to C24, C12 to C25, C11 to C26, C9 to C27, C30 to C28, C28 to C29, C29 to C30, C26 to C9, R20 to R19, R23 to R20, R19 to R21, R21 to R23, R25 to R24, R24 to R25, TP1 to TP3, TP3 to TP4, TP2 to TP5, U1 to U3

Commit message: Add Main Unit to CI build as well
Parts:
- C10, C15, C17, C18, C20, C23, C24, C27, C29: LibRef (none) -> ESD35C104K4T2A-24
- C11, C12, C13, C16, C21, C22, C25, C26, C28, C30, C9: LibRef (none) -> CL10B105MO8NNWC
- R19, R20, R21, R22, R23: LibRef (none) -> RC0603FR-0710KL
- R24, R25: LibRef (none) -> ERJ-3EKF33R0V
