File: hardware/Common Sheets/5V_To_3.3V_LDO.kicad_sch (KiCad schematic)
At the start: 3 parts, among them U2 TLV71333PDBV

Commit message: Oops forgot to save
Parts:
- C3, C4, U2: KiLib_Generator (none) -> Digi-Key
Changed lines of the file:
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@@
+			)
+		)
+		(property "KiLib_Generator" "Digi-Key"
+			(at 74.93 53.34 0)
+			(hide yes)
+			(show_name no)
+			(do_not_autoplace no)
+			(effects
+				(font
+					(size 1.27 1.27)
+				)
 			)
 		)
@@
 			)
 		)
+		(property "KiLib_Generator" "Digi-Key"
+			(at 87.63 55.88 0)
+			(hide yes)
+			(show_name no)
+			(do_not_autoplace no)
+			(effects
+				(font
+					(size 1.27 1.27)
+				)
+			)
+		)
 		(pin "1"
 		)
@@
 			(at 57.15 59.69 0)
 			(hide yes)
+			(show_name no)
+			(do_not_autoplace no)
+			(effects
+				(font
+					(size 1.27 1.27)
+				)
+			)
+		)
+		(property "KiLib_Generator" "Digi-Key"
+			(at 57.15 59.69 0)
+			(hide yes)

Commit message: Update voltage card to KiCAD 10
Parts:
- C14: renamed from C3; KiLib_Generator Digi-Key -> (none)
- C19: renamed from C4; KiLib_Generator Digi-Key -> (none)
- U2: KiLib_Generator Digi-Key -> (none)
Changed lines of the file:
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@@
-			)
-		)
-		(property "KiLib_Generator" "Digi-Key"
-			(at 74.93 53.34 0)
-			(hide yes)
-			(show_name no)
-			(do_not_autoplace no)
-			(effects
-				(font
-					(size 1.27 1.27)
-				)
 			)
 		)
@@
 		(dnp no)
 		(fields_autoplaced yes)
-		(property "Reference" "C3"
+		(property "Reference" "C14"
 			(at 90.17 54.6162 0)
 			(show_name no)
@@
 		)
 		(property "LibRef" "CL10B105MO8NNWC"
-			(at 87.63 55.88 0)
-			(hide yes)
-			(show_name no)
-			(do_not_autoplace no)
-			(effects
-				(font
-					(size 1.27 1.27)
-				)
-			)
-		)
-		(property "KiLib_Generator" "Digi-Key"
 			(at 87.63 55.88 0)
 			(hide yes)
@@
 		(dnp no)
 		(fields_autoplaced yes)
-		(property "Reference" "C4"
+		(property "Reference" "C19"
 			(at 59.69 58.4262 0)
 			(show_name no)
@@
 			(at 57.15 59.69 0)
 			(hide yes)
-			(show_name no)
-			(do_not_autoplace no)
-			(effects
-				(font
-					(size 1.27 1.27)
-				)
-			)
-		)
-		(property "KiLib_Generator" "Digi-Key"
-			(at 57.15 59.69 0)
-			(hide yes)
