File: hardware/Voltage Card/HackerDAQ Voltage Card.kicad_pcb (KiCad board)
At the start: 2 copper layers, 90 x 90 mm, 92 parts, among them J1 0039301040, J2 0039301040, J3 0039301040, J4 0039301040, J5 0039301040, J6 0039301040, J7 0039301040, J8 0039301040, J9 LD15S33E4GX00LF, U1 OPA310xDBV, U2 TLV71333PDBV, U3 AD7770, U4 M95320-RMN6

Commit message: Designator conflict :(
Parts:
- renumbered C5 to C31, C31 to C5, J9 to J6, J6 to J9, R26 to R33, U4 to U9
