File: hardware/Voltage Card/HackerDAQ Voltage Card.kicad_sch (KiCad schematic)
At the start: 22 parts, among them J1 0039301040, J2 0039301040, J3 0039301040, J4 0039301040, J5 0039301040, J6 0039301040, J7 0039301040, J8 0039301040, U1 OPA310xDBV

Commit message: Designator conflict :(
Parts:
- renumbered J6 to J9
Changed lines of the file:
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@@
 		(dnp no)
 		(fields_autoplaced yes)
-		(property "Reference" "J6"
+		(property "Reference" "J9"
 			(at 28.956 129.54 0)
 			(effects
@@
 			(project "HackerDAQ Voltage Card"
 				(path "/af2d881c-6553-449d-9093-6deb41497bdc"
-					(reference "J6")
+					(reference "J9")
 					(unit 1)
 				)

Commit message: Update voltage card to KiCAD 10
Parts:
- LG1: value ~ -> (none)
